File: kicad/audioout.sch (KiCad schematic (older format))
At the start: 67 parts

Commit message: ...
Parts:
- removed L?: bead, symbol L_Small
- added C406, C407: 0.39, symbol C_Small
- added C412, C413: 1.0, symbol C_Small
- added C414, C415, C?: 1nF, symbol C_Small
- added C420, C421: 0.1, symbol C_Small
- added C422, C423, C?: 4.7, symbol CP1_Small
- added C428, C429: 10.0, symbol CP1_Small
- added J401: ST-214N, symbol JACK_TRS_6PINS
- added L401, L402, L403: BLM21PG331SN1D, symbol L_Small
- added R427, R428: 20K, symbol R
- added R431, R436: 10K, symbol R
- added U403, U404: LM4864, symbol LM4864
- gave numbers to parts that had none: 63
Connections:
- net +12VOPA: now also C?.1, C?.1, L401.1
- net at C401.1, R401.1, R402.2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: now also L401.2
- net SE_LEFT: now reaches C438.1, J402.2 (T), R432.2, R434.1
- net SE_LEFT: now also C406.2
- net SE_RIGHT: now reaches C439.1, J402.3 (R), R433.2, R435.1
- net SE_RIGHT: now also C407.2
- net LINEOUT_PLUGGED: now reaches J402.4 (SN)
- net LINEOUT_PLUGGED: now also R436.2
- new net: C412.1, C414.1, U403.2 (BYPASS), U403.3 (+IN)
- new net: C406.1, R427.2, U403.4 (-IN)
- new net: R427.1, U403.5 (Vo1)
- new net: C428.1, U403.8 (Vo2)
- new net: C413.1, C415.1, U404.2 (BYPASS), U404.3 (+IN)
- new net: C407.1, R428.2, U404.4 (-IN)
- new net: R428.1, U404.5 (Vo1)
- new net: C429.1, U404.8 (Vo2)
- new net: J401.2 (T), L402.2
- new net: J401.3 (R), L403.2
- new net: C429.2, L403.1
- new net: C428.2, L402.1
- new net: C?.2, C?.2
- new net +3V3D_CPU: R436.1
- new net +5V_JACK: C420.1, C421.1, C422.1, C423.1, R431.2, U403.6 (Vdd), U404.6 (Vdd)
- new net GNDD: C412.2, C413.2, C414.2, C415.2, C420.2, C421.2, C422.2, C423.2, J401.1 (S), U403.7 (GND), U404.7 (GND)
- new net ~SHUTDOWN: J401.4 (SN), R431.1, U403.1 (~SHUTDOWN), U404.1 (~SHUTDOWN)
Other:
- note removed: "Detect plugged jack to start power supplies"
- moved on the sheet: C401, C402, C403, C404, C405, C408, C409, C410, C411, C416, C417, C418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

Commit message: ...
Parts:
- removed C423: 4.7, symbol CP1_Small
- added L?: BLM21PG331SN1D, symbol L_Small
- C422: value 4.7 -> 22.0
Connections:
- net +5V_JACK: now also L?.1; no longer C420.1, C421.1, C422.1, U403.6 (Vdd), U404.6 (Vdd)
- new net +5VHEAD: C420.1, C421.1, C422.1, L?.2, U403.6 (Vdd), U404.6 (Vdd)
Other:
- note removed: "Add headphone amplifier"
- moved on the sheet: C420, C421, C422
Changed lines of the file:
@@
 LIBS:ad1955
 LIBS:lm4864
+LIBS:mc33269
 LIBS:synth-cache
 EELAYER 25 0
@@
 	3300 2100 3300 1550
 Wire Wire Line
-	3300 1550 7450 1550
+	3300 1550 4300 1550
+Wire Wire Line
+	4300 1550 7450 1550
 Wire Wire Line
 	7450 1550 7700 1550
@@
 Connection ~ 7450 1850
 Connection ~ 6600 4100
-Text Notes 9800 5000 0    60   ~ 0
-Add headphone amplifier
 $Comp
 L LM4864 U403
@@
 $EndComp
 Wire Wire Line
-	5050 9000 5050 9450
-Wire Wire Line
-	5050 9450 5050 9700
-Wire Wire Line
-	5050 9700 5050 9800
+	5050 9500 5050 9550
+Wire Wire Line
+	5050 9550 5050 9800
 Wire Wire Line
 	4950 11400 5050 11400
 Wire Wire Line
-	5050 11400 5200 11400
-Wire Wire Line
-	5200 11400 5400 11400
+	5050 11400 5500 11400
 $Comp
 L C_Small C414
@@
 L C_Small C421
 U 1 1 567B798F
-P 5200 11550
-F 0 "C421" H 5210 11620 50  0000 L CNN
-F 1 "0.1" H 5210 11470 50  0000 L CNN
-F 2 "" H 5200 11550 50  0000 C CNN
-F 3 "" H 5200 11550 50  0000 C CNN
-	1    5200 11550
-	-1   0    0    -1
-$EndComp
-$Comp
-L CP1_Small C423
-U 1 1 567B7995
-P 5400 11550
-F 0 "C423" H 5410 11620 50  0000 L CNN
-F 1 "4.7" H 5410 11470 50  0000 L CNN
-F 2 "" H 5400 11550 50  0000 C CNN
-F 3 "" H 5400 11550 50  0000 C CNN
-	1    5400 11550
-	1    0    0    -1
-$EndComp
-Wire Wire Line
-	5200 11400 5200 11450
-Wire Wire Line
-	5400 11400 5400 11450
+P 5500 11550
+F 0 "C421" H 5510 11620 50  0000 L CNN
+F 1 "0.1" H 5510 11470 50  0000 L CNN
+F 2 "" H 5500 11550 50  0000 C CNN
+F 3 "" H 5500 11550 50  0000 C CNN
+	1    5500 11550
+	-1   0    0    -1
+$EndComp
+Wire Wire Line
+	5500 11400 5500 11450
 $Comp
 L GNDD #PWR068
 U 1 1 567B79A0
-P 5300 11650
-F 0 "#PWR068" H 5300 11400 50  0001 C CNN
-F 1 "GNDD" H 5300 11500 39  0000 C CNN
-F 2 "" H 5300 11650 50  0000 C CNN
-F 3 "" H 5300 11650 50  0000 C CNN
-	1    5300 11650
-	1    0    0    -1
-$EndComp
-Connection ~ 5200 11400
+P 5500 11650
+F 0 "#PWR068" H 5500 11400 50  0001 C CNN
+F 1 "GNDD" H 5500 11500 39  0000 C CNN
+F 2 "" H 5500 11650 50  0000 C CNN
+F 3 "" H 5500 11650 50  0000 C CNN
+	1    5500 11650
+	1    0    0    -1
+$EndComp
 $Comp
 L GNDD #PWR069
@@
 Wire Wire Line
 	4400 10200 4550 10200
-Connection ~ 5050 9700
 $Comp
 L JACK_TRS_6PINS J401
@@
 	4550 12450 4350 12450
 Wire Wire Line
-	5200 11650 5300 11650
-Wire Wire Line
-	5300 11650 5400 11650
-Connection ~ 5300 11650
-Connection ~ 5050 11400
-Wire Wire Line
-	5050 9450 5200 9450
-Wire Wire Line
-	5200 9450 5400 9450
+	5500 11650 5500 11650
+Wire Wire Line
+	3750 8700 4050 8700
+Wire Wire Line
+	4050 8700 4700 8700
 $Comp
 L C_Small C420
 U 1 1 567C90C2
-P 5200 9600
-F 0 "C420" H 5210 9670 50  0000 L CNN
-F 1 "0.1" H 5210 9520 50  0000 L CNN
-F 2 "" H 5200 9600 50  0000 C CNN
-F 3 "" H 5200 9600 50  0000 C CNN
-	1    5200 9600
-	-1   0    0    -1
+P 5500 9650
+F 0 "C420" H 5510 9720 50  0000 L CNN
+F 1 "0.1" H 5510 9570 50  0000 L CNN
+F 2 "" H 5500 9650 50  0000 C CNN
+F 3 "" H 5500 9650 50  0000 C CNN
+	1    5500 9650
+	1    0    0    -1
 $EndComp
 $Comp
 L CP1_Small C422
 U 1 1 567C90C8
-P 5400 9600
-F 0 "C422" H 5410 9670 50  0000 L CNN
-F 1 "4.7" H 5410 9520 50  0000 L CNN
-F 2 "" H 5400 9600 50  0000 C CNN
-F 3 "" H 5400 9600 50  0000 C CNN
-	1    5400 9600
-	1    0    0    -1
-$EndComp
-Wire Wire Line
-	5200 9450 5200 9500
-Wire Wire Line
-	5400 9450 5400 9500
+P 4050 8850
+F 0 "C422" H 4060 8920 50  0000 L CNN
+F 1 "22.0" H 4060 8770 50  0000 L CNN
+F 2 "" H 4050 8850 50  0000 C CNN
+F 3 "" H 4050 8850 50  0000 C CNN
+	1    4050 8850
+	1    0    0    -1
+$EndComp
+Wire Wire Line
+	4050 8700 4050 8750
 $Comp
 L GNDD #PWR076
 U 1 1 567C90D0
-P 5300 9700
-F 0 "#PWR076" H 5300 9450 50  0001 C CNN
-F 1 "GNDD" H 5300 9550 39  0000 C CNN
-F 2 "" H 5300 9700 50  0000 C CNN
-F 3 "" H 5300 9700 50  0000 C CNN
-	1    5300 9700
-	1    0    0    -1
-$EndComp
-Connection ~ 5200 9450
-Wire Wire Line
-	5200 9700 5300 9700
-Wire Wire Line
-	5300 9700 5400 9700
-Connection ~ 5300 9700
-Connection ~ 5050 9450
+P 4050 8950
+F 0 "#PWR076" H 4050 8700 50  0001 C CNN
+F 1 "GNDD" H 4050 8800 39  0000 C CNN
+F 2 "" H 4050 8950 50  0000 C CNN
+F 3 "" H 4050 8950 50  0000 C CNN
+	1    4050 8950
+	1    0    0    -1
+$EndComp
+Wire Wire Line
+	4050 8950 4050 8950
 Text Label 2850 10200 0    60   ~ 0
 ~SHUTDOWN
@@
 	0    -1   -1   0
 $EndComp
-Text GLabel 5050 9000 1    60   Input ~ 0
-+5V_JACK
-Text GLabel 4950 11400 0    60   Input ~ 0
+Text GLabel 3400 8700 0    60   Input ~ 0
 +5V_JACK
 Wire Wire Line
@@
 Connection ~ 4300 1750
 Connection ~ 4300 1550
+$Comp
+L L_Small L?
+U 1 1 568BB662
+P 3650 8700
+F 0 "L?" V 3750 8700 50  0000 L CNN
+F 1 "BLM21PG331SN1D" V 3850 8400 50  0000 L CNN
+F 2 "" H 3650 8700 50  0000 C CNN
+F 3 "" H 3650 8700 50  0000 C CNN
+	1    3650 8700
+	0    -1   -1   0
+$EndComp
+Wire Wire Line
+	3400 8700 3550 8700
+Connection ~ 4050 8700
+Text Label 4700 8700 2    60   ~ 0
++5VHEAD
+Text Label 5050 9500 2    60   ~ 0
++5VHEAD
+Wire Wire Line
+	5500 9550 5050 9550
+Connection ~ 5050 9550
+$Comp
+L GNDD #PWR?
+U 1 1 568C346E
+P 5500 9750
+F 0 "#PWR?" H 5500 9500 50  0001 C CNN
+F 1 "GNDD" H 5500 9600 39  0000 C CNN
+F 2 "" H 5500 9750 50  0000 C CNN
+F 3 "" H 5500 9750 50  0000 C CNN
+	1    5500 9750
+	1    0    0    -1
+$EndComp
+Text Label 4950 11400 0    60   ~ 0
++5VHEAD
+Connection ~ 5050 11400
 $EndSCHEMATC

Commit message: ...
Parts:
- removed J401, J402: ST-214N, symbol JACK_TRS_6PINS
- removed R431: 10K, symbol R
- added C301, C302: 0.01, Capacitors_SMD:C_0805, symbol C_Small
- added D301, D302: LED, LEDs:LED-0805, symbol LED
- added J301, J302: KATE_3.5MM_6, jacks:JACK_35MM_KATE_6, symbol KATE_3.5MM_6
- added P301: CONN_02X04, Pin_Headers:Pin_Header_Straight_2x04, symbol CONN_02X04
- added Q301: Si2301DS, TO_SOT_Packages_SMD:SOT-23, symbol Q_PMOS_GSD
- added R301, R302: 820, Resistors_SMD:R_0805, symbol R
- added R304: 470, Resistors_SMD:R_0805, symbol R
- added R339, R340: 10K, Resistors_SMD:R_0805, symbol R
- C303: renamed from C401; footprint (none) -> Capacitors_SMD:C_0805
- C304: renamed from C402; footprint (none) -> Capacitors_SMD:C_0805
- C305: renamed from C403; footprint (none) -> Capacitors_SMD:C_0805
- C306: renamed from C404; footprint (none) -> Capacitors_SMD:C_0805
- C307: renamed from C405; footprint (none) -> Capacitors_SMD:C_0805
- C308: renamed from C406; footprint (none) -> Capacitors_SMD:C_0805
- C309: renamed from C407; footprint (none) -> Capacitors_SMD:C_0805
- C310: renamed from C408; footprint (none) -> Capacitors_SMD:C_0805
- C311: renamed from C409; footprint (none) -> Capacitors_SMD:C_0805
- C312: renamed from C410; footprint (none) -> Capacitors_SMD:C_0805
- C313: renamed from C411; footprint (none) -> Capacitors_SMD:C_0805
- C314: renamed from C412; footprint (none) -> Capacitors_SMD:C_0805
- C315: renamed from C422; footprint (none) -> Capacitors_Tantalum_SMD:TantalC_SizeC_EIA-6032_Reflow
- C316: renamed from C413; footprint (none) -> Capacitors_SMD:C_0805
- C317: renamed from C414; footprint (none) -> Capacitors_SMD:C_0805
- C318, C320: renamed from C?; footprint (none) -> Capacitors_SMD:C_0805
- C319: renamed from C415; footprint (none) -> Capacitors_SMD:C_0805
- C321: renamed from C416; footprint (none) -> Capacitors_SMD:C_0805
- C322: renamed from C417; footprint (none) -> Capacitors_SMD:C_0805
- C323: renamed from C418; footprint (none) -> Capacitors_SMD:C_0805
- C324: renamed from C419; footprint (none) -> Capacitors_SMD:C_0805
- C325: renamed from C424; footprint (none) -> Capacitors_SMD:C_0805
- C326: renamed from C425; footprint (none) -> Capacitors_SMD:C_0805
- C327: renamed from C426; footprint (none) -> Capacitors_SMD:C_0805
- C328: renamed from C427; footprint (none) -> Capacitors_SMD:C_0805
- C329: renamed from C420; footprint (none) -> Capacitors_SMD:C_0805
- C330: renamed from C421; footprint (none) -> Capacitors_SMD:C_0805
- C331: renamed from C428; value 10.0 -> 22.0; footprint (none) -> Capacitors_Tantalum_SMD:TantalC_SizeC_EIA-6032_Reflow
- C332: renamed from C429; value 10.0 -> 22.0; footprint (none) -> Capacitors_Tantalum_SMD:TantalC_SizeC_EIA-6032_Reflow
- C333: renamed from C430; footprint (none) -> Capacitors_SMD:C_0805
- C334: renamed from C431; footprint (none) -> Capacitors_SMD:C_0805
- C335: renamed from C432; footprint (none) -> Capacitors_SMD:C_0805
- C336: renamed from C433; footprint (none) -> Capacitors_SMD:C_0805
- C337: renamed from C434; footprint (none) -> Capacitors_SMD:C_0805
- C338: renamed from C435; footprint (none) -> Capacitors_SMD:C_0805
- C339: renamed from C436; footprint (none) -> Capacitors_SMD:C_0805
- C340: renamed from C437; footprint (none) -> Capacitors_SMD:C_0805
- C341: renamed from C438; footprint (none) -> Capacitors_SMD:C_0805
- C342: renamed from C439; footprint (none) -> Capacitors_SMD:C_0805
- L301: renamed from L401; footprint (none) -> Resistors_SMD:R_0805
- L302: renamed from L?; footprint (none) -> Resistors_SMD:R_0805
- L303: renamed from L402; footprint (none) -> Resistors_SMD:R_0805
- L304: renamed from L403; footprint (none) -> Resistors_SMD:R_0805
- R305: renamed from R401; footprint (none) -> Resistors_SMD:R_0805
- R306: renamed from R402; footprint (none) -> Resistors_SMD:R_0805
- R307: renamed from R403; footprint (none) -> Resistors_SMD:R_0805
- R308: renamed from R404; footprint (none) -> Resistors_SMD:R_0805
- R309: renamed from R405; footprint (none) -> Resistors_SMD:R_0805
- R310: renamed from R406; footprint (none) -> Resistors_SMD:R_0805
- R311: renamed from R407; footprint (none) -> Resistors_SMD:R_0805
- R312: renamed from R408; footprint (none) -> Resistors_SMD:R_0805
- R313: renamed from R409; footprint (none) -> Resistors_SMD:R_0805
- R314: renamed from R410; footprint (none) -> Resistors_SMD:R_0805
- R315: renamed from R411; footprint (none) -> Resistors_SMD:R_0805
- R316: renamed from R412; footprint (none) -> Resistors_SMD:R_0805
- R317: renamed from R413; footprint (none) -> Resistors_SMD:R_0805
- R318: renamed from R414; footprint (none) -> Resistors_SMD:R_0805
- R319: renamed from R415; footprint (none) -> Resistors_SMD:R_0805
- R320: renamed from R416; footprint (none) -> Resistors_SMD:R_0805
- R321: renamed from R417; footprint (none) -> Resistors_SMD:R_0805
- R322: renamed from R418; footprint (none) -> Resistors_SMD:R_0805
- R323: renamed from R419; footprint (none) -> Resistors_SMD:R_0805
- R324: renamed from R420; footprint (none) -> Resistors_SMD:R_0805
- R325: renamed from R421; footprint (none) -> Resistors_SMD:R_0805
- R326: renamed from R422; footprint (none) -> Resistors_SMD:R_0805
- R327: renamed from R423; footprint (none) -> Resistors_SMD:R_0805
- R328: renamed from R424; footprint (none) -> Resistors_SMD:R_0805
- R329: renamed from R425; footprint (none) -> Resistors_SMD:R_0805
- R330: renamed from R426; footprint (none) -> Resistors_SMD:R_0805
- R331: renamed from R427; footprint (none) -> Resistors_SMD:R_0805
- R332: renamed from R428; footprint (none) -> Resistors_SMD:R_0805
- R333: renamed from R429; footprint (none) -> Resistors_SMD:R_0805
- R334: renamed from R430; footprint (none) -> Resistors_SMD:R_0805
- R335: renamed from R432; footprint (none) -> Resistors_SMD:R_0805
- R336: renamed from R433; footprint (none) -> Resistors_SMD:R_0805
- R337: renamed from R434; footprint (none) -> Resistors_SMD:R_0805
- R338: renamed from R435; footprint (none) -> Resistors_SMD:R_0805
- R341: renamed from R436; value 10K -> 47K; footprint (none) -> Resistors_SMD:R_0805
- U301: renamed from U401; footprint (none) -> Housings_SOIC:SOIC-8_3.9x4.9mm_Pitch1.27mm
- U302: renamed from U402; footprint (none) -> Housings_SOIC:SOIC-8_3.9x4.9mm_Pitch1.27mm
- U303: renamed from U403; footprint (none) -> Housings_SOIC:SOIC-8_3.9x4.9mm_Pitch1.27mm
- U304: renamed from U404; footprint (none) -> Housings_SOIC:SOIC-8_3.9x4.9mm_Pitch1.27mm
- U305: renamed from U405; footprint (none) -> Housings_SOIC:SOIC-8_3.9x4.9mm_Pitch1.27mm
Connections:
- net +5VHEAD: now also Q301.3 (D), R340.1
- net GNDA: now also C301.2, C302.1, D302.1 (K), J302.2 (S2), J302.3
- net GNDD: now also D301.1 (K), J301.2 (S2), J301.3
- net SE_LEFT: now also J302.6 (T), P301.1 (P1); no longer C308.2
- net SE_RIGHT: now also J302.5 (R), P301.3 (P3); no longer C309.2
- net ~SHUTDOWN: now also J301.1 (S1), J301.4 (S3), Q301.1 (G), R340.2
- net at L303.2: now also J301.6 (T)
- net at L304.2: now also J301.5 (R)
- net +3V3D_CPU renamed +3V3A_CPU
- net +5V_JACK renamed +5VJACK
- net LINEOUT_PLUGGED renamed LINEOUT_SW
- net LINEOUT_SW: now also J302.1 (S1), J302.4 (S3)
- new net: Q301.2 (S), R304.1
- new net: C308.2, P301.2 (P2), P301.6 (P6)
- new net: C309.2, P301.4 (P4), P301.8 (P8)
- new net: D301.2 (A), R304.2
- new net: D302.2 (A), R339.2
- new net: C301.1, P301.5 (P5), R301.2
- new net: C302.2, P301.7 (P7), R302.2
- new net +5VA_DAC: R339.1
- new net LF_LEFT: R301.1
- new net LF_RIGHT: R302.1
Other:
- note added: "5-pole (6-pin) 3.5mm Kate\nRegular 3.5mm Jack shorts out S1, S2, S3"
- moved on the sheet: R341

Commit message: before moving headphone amp to the left
Parts:
- added P302: CONN_01X03, Pin_Headers:Pin_Header_Straight_1x03, symbol CONN_01X03
- R301, R302, R307, R308: footprint Resistors_SMD:R_0805 -> Resistors_SMD:R_1206
Connections:
- net GNDA: now also C318.2, C320.2, C321.2, C322.2, C323.2, C324.2, C336.2, C338.2, C339.2, C340.2, P302.2 (P2)
- net SE_LEFT: now also P302.1 (P1)
- net SE_RIGHT: now also P302.3 (P3)
- net ~SHUTDOWN renamed PHONES_SW
Changed lines of the file:
@@
 F 0 "R307" V 2450 2300 50  0000 C CNN
 F 1 "402.0" V 2250 2300 50  0000 C CNN
-F 2 "Resistors_SMD:R_0805" V 2280 2300 50  0001 C CNN
+F 2 "Resistors_SMD:R_1206" V 2280 2300 50  0001 C CNN
 F 3 "" H 2350 2300 50  0000 C CNN
 	1    2350 2300
@@
 F 0 "R308" V 2430 6400 50  0000 C CNN
 F 1 "402.0" V 2250 6400 50  0000 C CNN
-F 2 "Resistors_SMD:R_0805" V 2280 6400 50  0001 C CNN
+F 2 "Resistors_SMD:R_1206" V 2280 6400 50  0001 C CNN
 F 3 "" H 2350 6400 50  0000 C CNN
 	1    2350 6400
@@
 F 0 "R301" V 1450 11300 50  0000 C CNN
 F 1 "820" V 1250 11300 50  0000 C CNN
-F 2 "Resistors_SMD:R_0805" V 1280 11300 50  0001 C CNN
+F 2 "Resistors_SMD:R_1206" V 1280 11300 50  0001 C CNN
 F 3 "" H 1350 11300 50  0000 C CNN
 	1    1350 11300
@@
 F 0 "R302" V 1450 12000 50  0000 C CNN
 F 1 "820" V 1250 12000 50  0000 C CNN
-F 2 "Resistors_SMD:R_0805" V 1280 12000 50  0001 C CNN
+F 2 "Resistors_SMD:R_1206" V 1280 12000 50  0001 C CNN
 F 3 "" H 1350 12000 50  0000 C CNN
 	1    1350 12000
@@
 Connection ~ 10050 4050
 Connection ~ 10150 4150
+$Comp
+L CONN_01X03 P302
+U 1 1 5676CE02
+P 9150 4300
+F 0 "P302" H 9150 4500 50  0000 C CNN
+F 1 "CONN_01X03" V 9300 4300 50  0000 C CNN
+F 2 "Pin_Headers:Pin_Header_Straight_1x03" H 9150 4300 50  0001 C CNN
+F 3 "" H 9150 4300 50  0000 C CNN
+	1    9150 4300
+	1    0    0    -1
+$EndComp
+Wire Wire Line
+	8950 4200 8950 2750
+Connection ~ 8950 2750
+Wire Wire Line
+	8950 4400 8950 5950
+Connection ~ 8950 5950
+$Comp
+L GNDA #PWR097
+U 1 1 5676D2E6
+P 8800 4300
+F 0 "#PWR097" H 8800 4050 50  0001 C CNN
+F 1 "GNDA" H 8800 4150 39  0000 C CNN
+F 2 "" H 8800 4300 50  0000 C CNN
+F 3 "" H 8800 4300 50  0000 C CNN
+	1    8800 4300
+	0    1    1    0
+$EndComp
+Wire Wire Line
+	8800 4300 8950 4300
+Connection ~ 6600 4500
+Connection ~ 4500 4900
+Connection ~ 4300 2050
+Connection ~ 7450 2300
+Connection ~ 4500 3650
+Wire Wire Line
+	8400 10700 8400 10500
+Wire Wire Line
+	8400 10500 8500 10500
+Connection ~ 8400 10700
+Text HLabel 8500 10500 2    60   Input ~ 0
+PHONES_SW
 $EndSCHEMATC

Commit message: gruuuu
Parts:
- added Q302: BC817, TO_SOT_Packages_SMD:SOT-23, symbol Q_NPN_BEC
- added R303: 1K, Resistors_SMD:R_0805, symbol R
- added R342: 10K, Resistors_SMD:R_0805, symbol R
Connections:
- net GNDD: now also Q302.2 (E)
- net IOUTL+: now also C304.1, R309.2, R311.1, R318.1, U301.2 (-); no longer C304.2, R305.2, R312.1, R315.1, U301.6 (-)
- net IOUTL-: now also C304.2, R305.2, R312.1, R315.1, U301.6 (-); no longer C304.1, R309.2, R311.1, R318.1, U301.2 (-)
- net PHONES_SW: now also Q302.3 (C), R342.2; no longer J301.1 (S1), J301.4 (S3), Q301.1 (G), R340.2, U303.1 (~SHUTDOWN), U304.1 (~SHUTDOWN)
- net at C326.2, R324.1, R328.1: now also R319.2; no longer R320.2
- net at C325.1, R323.2, R327.1: now also R320.2; no longer R319.2
- new net: Q302.1 (B), R303.1
- new net +3V3D_CPU: R342.1
- new net ~SHUTDOWN: J301.1 (S1), J301.4 (S3), Q301.1 (G), R303.2, R340.2, U303.1 (~SHUTDOWN), U304.1 (~SHUTDOWN)
