File: kicad/audioout.sch (KiCad schematic (older format))
At the start: 101 parts, among them J301 KATE_3.5MM_6, J302 KATE_3.5MM_6, P301 CONN_02X04, P302 CONN_01X03, Q301 Si2301DS, Q302 BC817, U301 OP275S, U302 OP275S, U303 LM4864, U304 LM4864, U305 OP275S

Commit message: drc ok large vias
Connections:
- net GNDA: no longer C301.2, C302.1
- net GNDD: now also C301.2, C302.1
Changed lines of the file:
@@
 $EndComp
 $Comp
-L GNDA #PWR302
+L GNDA #PWR066
 U 1 1 567835C0
 P 2000 4600
-F 0 "#PWR302" H 2000 4350 50  0001 C CNN
+F 0 "#PWR066" H 2000 4350 50  0001 C CNN
 F 1 "GNDA" H 2000 4450 39  0000 C CNN
 F 2 "" H 2000 4600 50  0000 C CNN
@@
 $EndComp
 $Comp
-L GNDA #PWR314
+L GNDA #PWR067
 U 1 1 5678AFA5
 P 5100 2800
-F 0 "#PWR314" H 5100 2550 50  0001 C CNN
+F 0 "#PWR067" H 5100 2550 50  0001 C CNN
 F 1 "GNDA" H 5100 2650 39  0000 C CNN
 F 2 "" H 5100 2800 50  0000 C CNN
@@
 $EndComp
 $Comp
-L GNDA #PWR318
+L GNDA #PWR068
 U 1 1 5678C0A4
 P 6400 1800
-F 0 "#PWR318" H 6400 1550 50  0001 C CNN
+F 0 "#PWR068" H 6400 1550 50  0001 C CNN
 F 1 "GNDA" H 6400 1650 39  0000 C CNN
 F 2 "" H 6400 1800 50  0000 C CNN
@@
 $EndComp
 $Comp
-L GNDA #PWR323
+L GNDA #PWR069
 U 1 1 5678CF99
 P 8050 3200
-F 0 "#PWR323" H 8050 2950 50  0001 C CNN
+F 0 "#PWR069" H 8050 2950 50  0001 C CNN
 F 1 "GNDA" H 8050 3050 39  0000 C CNN
 F 2 "" H 8050 3200 50  0000 C CNN
@@
 $EndComp
 $Comp
-L GNDA #PWR325
+L GNDA #PWR070
 U 1 1 5678D24D
 P 8550 3200
-F 0 "#PWR325" H 8550 2950 50  0001 C CNN
+F 0 "#PWR070" H 8550 2950 50  0001 C CNN
 F 1 "GNDA" H 8550 3050 39  0000 C CNN
 F 2 "" H 8550 3200 50  0000 C CNN
@@
 $EndComp
 $Comp
-L GNDA #PWR315
+L GNDA #PWR071
 U 1 1 5678F030
 P 5100 5900
-F 0 "#PWR315" H 5100 5650 50  0001 C CNN
+F 0 "#PWR071" H 5100 5650 50  0001 C CNN
 F 1 "GNDA" H 5100 5750 39  0000 C CNN
 F 2 "" H 5100 5900 50  0000 C CNN
@@
 $EndComp
 $Comp
-L GNDA #PWR319
+L GNDA #PWR072
 U 1 1 5678F065
 P 6500 6900
-F 0 "#PWR319" H 6500 6650 50  0001 C CNN
+F 0 "#PWR072" H 6500 6650 50  0001 C CNN
 F 1 "GNDA" H 6500 6750 39  0000 C CNN
 F 2 "" H 6500 6900 50  0000 C CNN
@@
 $EndComp
 $Comp
-L GNDA #PWR324
+L GNDA #PWR073
 U 1 1 5678F096
 P 8050 5500
-F 0 "#PWR324" H 8050 5250 50  0001 C CNN
+F 0 "#PWR073" H 8050 5250 50  0001 C CNN
 F 1 "GNDA" H 8050 5350 39  0000 C CNN
 F 2 "" H 8050 5500 50  0000 C CNN
@@
 $EndComp
 $Comp
-L GNDA #PWR326
+L GNDA #PWR074
 U 1 1 5678F0A4
 P 8550 5500
-F 0 "#PWR326" H 8550 5250 50  0001 C CNN
+F 0 "#PWR074" H 8550 5250 50  0001 C CNN
 F 1 "GNDA" H 8550 5350 39  0000 C CNN
 F 2 "" H 8550 5500 50  0000 C CNN
@@
 $EndComp
 $Comp
-L GNDA #PWR330
+L GNDA #PWR075
 U 1 1 56794DA8
 P 9900 4150
-F 0 "#PWR330" H 9900 3900 50  0001 C CNN
+F 0 "#PWR075" H 9900 3900 50  0001 C CNN
 F 1 "GNDA" H 9900 4000 39  0000 C CNN
 F 2 "" H 9900 4150 50  0000 C CNN
@@
 $EndComp
 $Comp
-L GNDA #PWR321
+L GNDA #PWR076
 U 1 1 567967A1
 P 7450 2300
-F 0 "#PWR321" H 7450 2050 50  0001 C CNN
+F 0 "#PWR076" H 7450 2050 50  0001 C CNN
 F 1 "GNDA" H 7450 2150 39  0000 C CNN
 F 2 "" H 7450 2300 50  0000 C CNN
@@
 $EndComp
 $Comp
-L GNDA #PWR310
+L GNDA #PWR077
 U 1 1 56799D3B
 P 4500 3650
-F 0 "#PWR310" H 4500 3400 50  0001 C CNN
+F 0 "#PWR077" H 4500 3400 50  0001 C CNN
 F 1 "GNDA" H 4500 3500 39  0000 C CNN
 F 2 "" H 4500 3650 50  0000 C CNN
@@
 $EndComp
 $Comp
-L GNDA #PWR303
+L GNDA #PWR078
 U 1 1 5679C52D
 P 3300 7650
-F 0 "#PWR303" H 3300 7400 50  0001 C CNN
+F 0 "#PWR078" H 3300 7400 50  0001 C CNN
 F 1 "GNDA" H 3300 7500 39  0000 C CNN
 F 2 "" H 3300 7650 50  0000 C CNN
@@
 $EndComp
 $Comp
-L GNDA #PWR311
+L GNDA #PWR079
 U 1 1 5679EC73
 P 4500 4900
-F 0 "#PWR311" H 4500 4650 50  0001 C CNN
+F 0 "#PWR079" H 4500 4650 50  0001 C CNN
 F 1 "GNDA" H 4500 4750 39  0000 C CNN
 F 2 "" H 4500 4900 50  0000 C CNN
@@
 $EndComp
 $Comp
-L GNDA #PWR320
+L GNDA #PWR080
 U 1 1 567A24C6
 P 6600 4500
-F 0 "#PWR320" H 6600 4250 50  0001 C CNN
+F 0 "#PWR080" H 6600 4250 50  0001 C CNN
 F 1 "GNDA" H 6600 4350 39  0000 C CNN
 F 2 "" H 6600 4500 50  0000 C CNN
@@
 $EndComp
 $Comp
-L GNDD #PWR317
+L GNDD #PWR081
 U 1 1 567B79A0
 P 5500 11650
-F 0 "#PWR317" H 5500 11400 50  0001 C CNN
+F 0 "#PWR081" H 5500 11400 50  0001 C CNN
 F 1 "GNDD" H 5500 11500 39  0000 C CNN
 F 2 "" H 5500 11650 50  0000 C CNN
@@
 $EndComp
 $Comp
-L GNDD #PWR312
+L GNDD #PWR082
 U 1 1 567B8574
 P 5050 11000
-F 0 "#PWR312" H 5050 10750 50  0001 C CNN
+F 0 "#PWR082" H 5050 10750 50  0001 C CNN
 F 1 "GNDD" H 5050 10850 39  0000 C CNN
 F 2 "" H 5050 11000 50  0000 C CNN
@@
 $EndComp
 $Comp
-L GNDD #PWR313
+L GNDD #PWR083
 U 1 1 567B9E9E
 P 5050 12950
-F 0 "#PWR313" H 5050 12700 50  0001 C CNN
+F 0 "#PWR083" H 5050 12700 50  0001 C CNN
 F 1 "GNDD" H 5050 12800 39  0000 C CNN
 F 2 "" H 5050 12950 50  0000 C CNN
@@
 $EndComp
 $Comp
-L GNDD #PWR322
+L GNDD #PWR084
 U 1 1 567BF38E
 P 7650 11200
-F 0 "#PWR322" H 7650 10950 50  0001 C CNN
+F 0 "#PWR084" H 7650 10950 50  0001 C CNN
 F 1 "GNDD" H 7650 11050 39  0000 C CNN
 F 2 "" H 7650 11200 50  0000 C CNN
@@
 $EndComp
 $Comp
-L GNDD #PWR307
+L GNDD #PWR085
 U 1 1 567C53BE
 P 4150 10900
-F 0 "#PWR307" H 4150 10650 50  0001 C CNN
+F 0 "#PWR085" H 4150 10650 50  0001 C CNN
 F 1 "GNDD" H 4150 10750 39  0000 C CNN
 F 2 "" H 4150 10900 50  0000 C CNN
@@
 $EndComp
 $Comp
-L GNDD #PWR304
+L GNDD #PWR086
 U 1 1 567C54B6
 P 3900 10900
-F 0 "#PWR304" H 3900 10650 50  0001 C CNN
+F 0 "#PWR086" H 3900 10650 50  0001 C CNN
 F 1 "GNDD" H 3900 10750 39  0000 C CNN
 F 2 "" H 3900 10900 50  0000 C CNN
@@
 $EndComp
 $Comp
-L GNDD #PWR306
+L GNDD #PWR087
 U 1 1 567C55AE
 P 4100 12900
-F 0 "#PWR306" H 4100 12650 50  0001 C CNN
+F 0 "#PWR087" H 4100 12650 50  0001 C CNN
 F 1 "GNDD" H 4100 12750 39  0000 C CNN
 F 2 "" H 4100 12900 50  0000 C CNN
@@
 $EndComp
 $Comp
-L GNDD #PWR309
+L GNDD #PWR088
 U 1 1 567C56A6
 P 4350 12900
-F 0 "#PWR309" H 4350 12650 50  0001 C CNN
+F 0 "#PWR088" H 4350 12650 50  0001 C CNN
 F 1 "GNDD" H 4350 12750 39  0000 C CNN
 F 2 "" H 4350 12900 50  0000 C CNN
@@
 $EndComp
 $Comp
-L GNDD #PWR305
+L GNDD #PWR089
 U 1 1 567C90D0
 P 4050 8950
-F 0 "#PWR305" H 4050 8700 50  0001 C CNN
+F 0 "#PWR089" H 4050 8700 50  0001 C CNN
 F 1 "GNDD" H 4050 8800 39  0000 C CNN
 F 2 "" H 4050 8950 50  0000 C CNN
@@
 $EndComp
 $Comp
-L GNDA #PWR308
+L GNDA #PWR090
 U 1 1 56863182
 P 4300 2050
-F 0 "#PWR308" H 4300 1800 50  0001 C CNN
+F 0 "#PWR090" H 4300 1800 50  0001 C CNN
 F 1 "GNDA" H 4300 1900 39  0000 C CNN
 F 2 "" H 4300 2050 50  0000 C CNN
@@
 +5VHEAD
 $Comp
-L GNDD #PWR316
+L GNDD #PWR091
 U 1 1 568C346E
 P 5500 9750
-F 0 "#PWR316" H 5500 9500 50  0001 C CNN
+F 0 "#PWR091" H 5500 9500 50  0001 C CNN
 F 1 "GNDD" H 5500 9600 39  0000 C CNN
 F 2 "" H 5500 9750 50  0000 C CNN
@@
 $EndComp
 $Comp
-L GNDA #PWR327
+L GNDA #PWR092
 U 1 1 569DDE27
 P 8600 7750
-F 0 "#PWR327" H 8600 7500 50  0001 C CNN
+F 0 "#PWR092" H 8600 7500 50  0001 C CNN
 F 1 "GNDA" H 8600 7600 39  0000 C CNN
 F 2 "" H 8600 7750 50  0000 C CNN
@@
 	1    0    0    -1
 $EndComp
-$Comp
-L GNDA #PWR301
-U 1 1 56A347AA
-P 1300 11650
-F 0 "#PWR301" H 1300 11400 50  0001 C CNN
-F 1 "GNDA" H 1300 11500 39  0000 C CNN
-F 2 "" H 1300 11650 50  0000 C CNN
-F 3 "" H 1300 11650 50  0000 C CNN
-	1    1300 11650
-	1    0    0    -1
-$EndComp
 Text Label 2000 11350 0    60   ~ 0
 SE_LEFT
@@
 	8950 10050 9000 10050
 $Comp
-L GNDD #PWR329
+L GNDD #PWR094
 U 1 1 567704E5
 P 9500 10200
-F 0 "#PWR329" H 9500 9950 50  0001 C CNN
+F 0 "#PWR094" H 9500 9950 50  0001 C CNN
 F 1 "GNDD" H 9500 10050 39  0000 C CNN
 F 2 "" H 9500 10200 50  0000 C CNN
@@
 Connection ~ 8950 5950
 $Comp
-L GNDA #PWR328
+L GNDA #PWR095
 U 1 1 5676D2E6
 P 8800 4300
-F 0 "#PWR328" H 8800 4050 50  0001 C CNN
+F 0 "#PWR095" H 8800 4050 50  0001 C CNN
 F 1 "GNDA" H 8800 4150 39  0000 C CNN
 F 2 "" H 8800 4300 50  0000 C CNN
@@
 	10500 10450 10500 10500
 $Comp
-L GNDD #PWR331
+L GNDD #PWR096
 U 1 1 567DAD9C
 P 10500 10900
-F 0 "#PWR331" H 10500 10650 50  0001 C CNN
+F 0 "#PWR096" H 10500 10650 50  0001 C CNN
 F 1 "GNDD" H 10500 10750 39  0000 C CNN
 F 2 "" H 10500 10900 50  0000 C CNN
@@
 	10500 10500 10800 10500
 Connection ~ 10500 10500
+$Comp
+L GNDD #PWR?
+U 1 1 56784490
+P 1300 11650
+F 0 "#PWR?" H 1300 11400 50  0001 C CNN
+F 1 "GNDD" H 1300 11500 39  0000 C CNN
+F 2 "" H 1300 11650 50  0000 C CNN
+F 3 "" H 1300 11650 50  0000 C CNN
+	1    1300 11650
+	1    0    0    -1
+$EndComp
 $EndSCHEMATC
