File: kicad/audioout.sch (KiCad schematic (older format))
At the start: 101 parts, among them J301 KATE_3.5MM_6, J302 KATE_3.5MM_6, P301 CONN_02X04, P302 CONN_01X03, Q301 Si2301DS, Q302 BC817, U301 OP275S, U302 OP275S, U303 LM4864, U304 LM4864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

Commit message: fixed p-mosfets
Parts:
- R339: value 10K -> 330
Connections:
- net +5VHEAD: now also Q301.2 (S); no longer Q301.3 (D)
- net at R304.1: now also Q301.3 (D); no longer Q301.2 (S)
Changed lines of the file:
@@
 P 8600 6700
 F 0 "R339" V 8700 6700 50  0000 C CNN
-F 1 "10K" V 8500 6700 50  0000 C CNN
+F 1 "330" V 8500 6700 50  0000 C CNN
 F 2 "Resistors_SMD:R_0805" V 8530 6700 50  0001 C CNN
 F 3 "" H 8600 6700 50  0000 C CNN
@@
 F 3 "" H 8250 10150 50  0000 C CNN
 	1    8250 10150
-	0    -1   -1   0
+	0    1    -1   0
 $EndComp
 Connection ~ 7800 10050
