File: kicad/synth.sch (KiCad schematic (older format))
At the start: 44 parts, among them P101 47346-0001, P102 DIN_5, U101 STM32F405R, U102 USBLC6-2, U103 AD1955, U104 HCPL0453, Y101 25MHz

Commit message: ...
Parts:
- removed RV101, RV102: PTD901-2015K-B103 10K, symbol POT
- added C? (x2): 0.1, symbol C_Small
- added C?: 22.0, symbol CP1_Small
- added CON?: SD_Card, 10067847-001, symbol SD_Card
- added D?: LED, symbol LED
- added P?: CONN_01X05, symbol CONN_01X05
- added P? (x2): CONN_01X03, symbol CONN_01X03
- added Q?: MMBTA42, symbol Q_NPN_BEC
- added R? (x3): 10K, symbol R_Small
- added R? (x4): 330, symbol R
- added R? (x3): 47K, symbol R
- added R?: 220, symbol R
- added R?: 1K, symbol R
- added SW? (x2): SW_PUSH, symbol SW_PUSH
Connections:
- net SPI_MISO is gone; now on net ~DAC_CS: U101.56 (PB4/NJTRST/SPI3_MISO/TIM3_CH1/SPI1_MISO/I2S3ext_SD)
- net +3V3D_CPU: now also C?.1, C?.1, CON?.4 (VDD), P?.1 (P1), R?.1, R?.2, R?.2, R?.2, R?.2, SW?.2
- net GNDD: now also BT101.2, C?.2, C?.2, C?.2, CON?.3 (VSS), CON?.6 (VSS), P?.3 (P3), Q?.2 (E), R?.1, R?.1, SW?.1
- net MIDI_RX: now also R?.1
- net PWM_FB: now also U101.14 (PA0/WKUP/USART2_CTS/UART4_TX/TIM2_CH1_ETR/TIM5_CH1/TIM8_ETR); no longer U101.26 (PB0/TIM3_CH3/TIM8_CH2N/OTG_HS_ULPI_D1/TIM1_CH2N)
- net UART3_TX: now also U101.51 (PC10/SPI3_SCK/I2S3_CK/UART4_TX/SDIO_D2/USART3_TX); no longer U101.29 (PB10/SPI2_SCK/I2S2_CK/I2C2_SCL/USART3_TX/OTG_HS_ULPI_D3/TIM2_CH3)
- net ~DAC_CS: no longer U101.52 (PC11/UART4_RX/SPI3_MISO/SDIO_D3/USART3_RX/I2S3ext_SD)
- net at U101.1 (VBAT): now also BT101.1, C?.1
- net ADC1_IN12_L: now reaches U101.10 (PC2/SPI2_MISO/OTG_HS_ULPI_DIR/I2S2ext_SD)
- net ADC2_IN13_R: now reaches U101.11 (PC3/SPI2_MOSI/I2S2_SD/OTG_HS_ULPI_NXT)
- net UART2_TX: now reaches U101.16 (PA2/USART2_TX/TIM5_CH3/TIM9_CH1/TIM2_CH3)
- net UART2_TX: now also R?.2
- net UART2_RX: now reaches U101.17 (PA3/USART2_RX/TIM5_CH4/TIM9_CH2/TIM2_CH4/OTG_HS_ULPI_D0)
- net UART2_RX: now also R?.2
- net PLUG1: now reaches U101.2 (PC13)
- net ADC1_IN6_HIGAIN1: now reaches U101.22 (PA6/SPI1_MISO/TIM8_BKIN/TIM13_CH1/TIM3_CH1/TIM1_BKIN)
- net ADC2_IN7_HIGAIN2: now reaches U101.23 (PA7/SPI1_MOSI/TIM8_CH1N/TIM14_CH1/TIM3_CH2/TIM1_CH1N)
- net at U101.28 (PB2/BOOT1): now also R?.2
- net PLUG2: now reaches U101.3 (PC14/OSC32_IN)
- net SDIO_D0: now reaches U101.39 (PC8/TIM8_CH3/SDIO_D0/TIM3_CH3/USART6_CK)
- net SDIO_D0: now also CON?.7 (DAT0), R?.1
- net PLUG3: now reaches U101.4 (PC15/OSC32_OUT)
- net LEDPLUG2: now reaches U101.40 (PC9/I2S_CKIN/MCO2/TIM8_CH4/SDIO_D1/I2C3_SDA/TIM3_CH4)
- net LEDPLUG3: now reaches U101.41 (PA8/MCO1/USART1_CK/TIM1_CH1/I2C3_SCL/OTG_FS_SOF)
- net SWDIO: now reaches U101.46 (PA13/JTMS/SWDIO)
- net SWDIO: now also P?.4 (P4)
- net SWCLK: now reaches U101.49 (PA14/JTCK/SWCLK)
- net SWCLK: now also P?.2 (P2)
- net SDIO_CK: now reaches U101.53 (PC12/UART5_TX/SDIO_CK/SPI3_MOSI/I2S3_SD/USART3_CK)
- net SDIO_CK: now also CON?.5 (CLK), R?.1
- net SDIO_CMD: now reaches U101.54 (PD2/TIM3_ETR/UART5_RX/SDIO_CMD)
- net SDIO_CMD: now also CON?.2 (CMD), R?.1
- net UART1_TX: now reaches U101.58 (PB6/I2C1_SCL/TIM4_CH1/CAN2_TX/USART1_TX)
- net UART1_TX: now also R?.2
- net UART1_RX: now reaches U101.59 (PB7/I2C1_SDA/FSMC_NL/USART1_RX/TIM4_CH2)
- net UART1_RX: now also R?.2
- net at U101.60 (BOOT0): now also R?.2, SW?.1
- net OUT_PLUGGED: now reaches U101.61 (PB8/TIM4_CH3/SDIO_D4/TIM10_CH1/I2C1_SCL/CAN1_RX)
- net ~RESET: now reaches U101.7 (NRST)
- net ~RESET: now also P?.5 (P5), R?.1, SW?.2
- net POT1: now reaches U101.8 (PC0/OTG_HS_ULPI_STP)
- net POT2: now reaches U101.9 (PC1)
- new net: P?.1 (P1), R?.1 (x2)
- new net: P?.2 (P2), R?.1 (x2)
- new net: Q?.1 (B), R?.2
- new net: D?.1 (K), Q?.3 (C)
- new net: D?.2 (A), R?.2
- new net LEDPLUG1: U101.52 (PC11/UART4_RX/SPI3_MISO/SDIO_D3/USART3_RX/I2S3ext_SD)
- no-connect marks 12 -> 19
Other:
- note added: "=ADC3_IN0"
- note added: "Pump feedback: ADC1_IN8\n\nADC dual mode inputs\npot inputs\nselector buttons\n\nchannel activity leds"
- note removed: "PWM Feedback: ADC1 CH8 (reassigned to PB0 @ pin 26)"
- moved on the sheet: BT101, C101, C102, C103, C104, C105, C106, C107, C108, C109, C110, R106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

Commit message: ...
Parts:
- added P105: CONN_01X01, SMD_Packages:1Pin, symbol CONN_01X01
- BT101: footprint CH25-2032(LF) -> ch25-2032LF:ch25-2032LF
- C101, C102, C103, C104, C108: footprint (none) -> Capacitors_SMD:C_0805
- C105, C106, C107: footprint (none) -> Capacitors_SMD:C_0603
- C109: renamed from C111; footprint (none) -> Capacitors_SMD:C_0805
- C110: renamed from C109; footprint (none) -> Capacitors_SMD:C_0603
- C111: renamed from C110; footprint (none) -> Capacitors_SMD:C_0805
- C112, C114: renamed from C?; footprint (none) -> Capacitors_SMD:C_0603
- C113: renamed from C112; footprint (none) -> Capacitors_SMD:C_0805
- C115: renamed from C?; footprint (none) -> Capacitors_Tantalum_SMD:TantalC_SizeD_EIA-7343_Reflow
- C116: renamed from C113; footprint (none) -> Capacitors_SMD:C_0805
- C117: renamed from C114; footprint (none) -> Capacitors_SMD:C_0805
- C118: renamed from C115; footprint (none) -> Capacitors_SMD:C_0805
- C119: renamed from C116; footprint (none) -> Capacitors_SMD:C_0805
- C120: renamed from C117; footprint (none) -> Capacitors_SMD:C_0603
- C121: renamed from C118; footprint (none) -> Capacitors_SMD:C_0805
- C122: renamed from C119; footprint (none) -> Capacitors_SMD:C_0603
- C123: renamed from C120; footprint (none) -> Capacitors_SMD:c_elec_5x5.3
- CON101: renamed from CON?; footprint 10067847-001 -> Connect:SD_Card_Receptacle
- D101: footprint (none) -> Diodes_SMD:SMB_Standard
- D102: footprint (none) -> TO_SOT_Packages_SMD:SOT-23
- D103: renamed from D?; footprint (none) -> LEDs:LED-0805
- L101, L102: footprint (none) -> Resistors_SMD:R_0805
- P101: renamed from P?; footprint (none) -> Pin_Headers:Pin_Header_Straight_1x05
- P102, P103: renamed from P?; footprint (none) -> Pin_Headers:Pin_Header_Straight_1x03
- P104: renamed from P101; footprint (none) -> Connect:USB_Micro-B
- P106: renamed from P102; footprint (none) -> w_conn_av:din-5
- Q101: renamed from Q?; footprint (none) -> TO_SOT_Packages_SMD:SOT-23
- R101, R102, R103, R104, R105, R106, R112, R113, R114, R115, R121, R122: renamed from R?; footprint (none) -> Resistors_SMD:R_0805
- R107: renamed from R101; footprint (none) -> Resistors_SMD:R_0805
- R108: renamed from R102; footprint (none) -> Resistors_SMD:R_0805
- R109: renamed from R103; footprint (none) -> Resistors_SMD:R_0805
- R110: renamed from R104; footprint (none) -> Resistors_SMD:R_0805
- R111: renamed from R105; footprint (none) -> Resistors_SMD:R_0805
- R116: renamed from R108; footprint (none) -> Resistors_SMD:R_0805
- R117: renamed from R106; footprint (none) -> Resistors_SMD:R_0402
- R118: renamed from R107; footprint (none) -> Resistors_SMD:R_0402
- R119: renamed from R109; footprint (none) -> Resistors_SMD:R_0805
- R120: renamed from R110; footprint (none) -> Resistors_SMD:R_0805
- SW101, SW102: renamed from SW?; footprint (none) -> Buttons_Switches_ThroughHole:SW_PUSH_SMALL
- U101: footprint TQFP64 -> Housings_QFP:TQFP-64_10x10mm_Pitch0.5mm
- U102: footprint (none) -> TO_SOT_Packages_SMD:SOT-23-6
- U103: footprint MODULE -> Housings_SSOP:SSOP-28_5.3x10.2mm_Pitch0.65mm
- U104: footprint SO8 -> Housings_SOIC:SOIC-8_3.9x4.9mm_Pitch1.27mm
- Y101: footprint HC-49SM -> Crystals:Crystal_HC49-SD_SMD
Connections:
- net GNDD: now also P102.3 (P3), P103.3 (P3)
- net UART3_TX: now also P105.1 (P1)
- net OUT_PLUGGED renamed LINEOUT_SW
- no-connect marks 19 -> 26
Other:
- moved on the sheet: C120, C121, C122, C123

Commit message: before moving headphone amp to the left
Connections:
- net PHONES_SW: now reaches U101.62 (PB9/SPI2_NSS/I2S2_WS/TIM4_CH4/TIM11_CH1/SDIO_D5/I2C1_SDA/CAN1_TX)
- no-connect marks 26 -> 25
Changed lines of the file:
@@
 F8 "LF_LEFT" I L 14950 6200 60
 F9 "LF_RIGHT" I L 14950 6350 60
+F10 "PHONES_SW" I L 14950 6000 60
 $EndSheet
 $Comp
@@
 $EndComp
 NoConn ~ 9000 5800
-NoConn ~ 9000 4200
+Wire Wire Line
+	14950 6000 14350 6000
+Text Label 14350 6000 0    60   ~ 0
+PHONES_SW
+Wire Wire Line
+	9000 4200 9750 4200
+Text Label 9750 4200 2    60   ~ 0
+PHONES_SW
 $EndSCHEMATC

Commit message: gruuuu
Connections:
- net LEDPLUG1: no longer names the net of U101.52 (PC11/UART4_RX/SPI3_MISO/SDIO_D3/USART3_RX/I2S3ext_SD)
- net LEDPLUG2: no longer names the net of U101.40 (PC9/I2S_CKIN/MCO2/TIM8_CH4/SDIO_D1/I2C3_SDA/TIM3_CH4)
- net LEDPLUG3: no longer names the net of U101.41 (PA8/MCO1/USART1_CK/TIM1_CH1/I2C3_SCL/OTG_FS_SOF)
- no-connect marks 25 -> 28
Changed lines of the file:
@@
 	11650 4600 11550 4600
-Wire Wire Line
-	9000 6200 9700 6200
 Wire Wire Line
 	2000 5700 1450 5700
@@
 F9 "PLUG_2" I R 2150 10150 60
 F10 "PLUG_3" I R 2150 10300 60
-F11 "LEDPLUG1" I L 1600 10500 60
-F12 "LEDPLUG2" I L 1600 10650 60
-F13 "LEDPLUG3" I L 1600 10800 60
 $EndSheet
 Wire Wire Line
@@
 Wire Wire Line
 	2150 10300 2600 10300
-Wire Wire Line
-	1600 10500 1100 10500
-Wire Wire Line
-	1600 10650 1100 10650
-Wire Wire Line
-	1600 10800 1100 10800
 Text Label 2600 10000 2    60   ~ 0
 PLUG1
@@
 Text Label 2600 10300 2    60   ~ 0
 PLUG3
-Text Label 1100 10500 0    60   ~ 0
-LEDPLUG1
-Text Label 1100 10650 0    60   ~ 0
-LEDPLUG2
-Text Label 1100 10800 0    60   ~ 0
-LEDPLUG3
 Wire Wire Line
 	2000 4800 1350 4800
@@
 Text Label 9700 6600 2    60   ~ 0
 PLUG3
-Text Label 9700 6200 2    60   ~ 0
-LEDPLUG1
-Wire Wire Line
-	9000 6000 9700 6000
-Text Label 9700 6000 2    60   ~ 0
-LEDPLUG2
-Wire Wire Line
-	2000 6000 1450 6000
-Text Label 1450 6000 0    60   ~ 0
-LEDPLUG3
 Wire Wire Line
 	14950 5850 14350 5850
@@
 Text Label 9750 4200 2    60   ~ 0
 PHONES_SW
+NoConn ~ 9000 6200
+NoConn ~ 9000 6000
+NoConn ~ 2000 6000
 $EndSCHEMATC

Commit message: battery is on the wrong side... sigh
Parts:
- added R? (x4): 47, Resistors_SMD:R_0402, symbol R
Connections:
- net I2S_CK: now also R?.2; no longer U101.34 (PB13/SPI2_SCK/I2S2_CK/USART3_CTS/TIM1_CH1N/CAN2_TX/OTG_HS_ULPI_D6)
- net I2S_MCK: now also R?.2; no longer U101.37 (PC6/I2S2_MCK/TIM8_CH1/SDIO_D6/USART6_TX/TIM3_CH1)
- net I2S_SD: now also R?.2; no longer U101.36 (PB15/SPI2_MOSI/I2S2_SD/TIM1_CH3N/TIM8_CH3N/TIM12_CH2/OTG_HS_DP)
- net I2S_WS: now also R?.2; no longer U101.33 (PB12/SPI2_NSS/I2S2_WS/I2C2_SMBA/USART3_CK/TIM1_BKIN/CAN2_RX/OTG_HS_ULPI_D5/OTG_HS_ID)
- new net I2S_CK#: R?.1, U101.34 (PB13/SPI2_SCK/I2S2_CK/USART3_CTS/TIM1_CH1N/CAN2_TX/OTG_HS_ULPI_D6)
- new net I2S_MCK#: R?.1, U101.37 (PC6/I2S2_MCK/TIM8_CH1/SDIO_D6/USART6_TX/TIM3_CH1)
- new net I2S_SD#: R?.1, U101.36 (PB15/SPI2_MOSI/I2S2_SD/TIM1_CH3N/TIM8_CH3N/TIM12_CH2/OTG_HS_DP)
- new net I2S_WS#: R?.1, U101.33 (PB12/SPI2_NSS/I2S2_WS/I2C2_SMBA/USART3_CK/TIM1_BKIN/CAN2_RX/OTG_HS_ULPI_D5/OTG_HS_ID)
Changed lines of the file:
@@
 $EndComp
 Text Label 9700 5700 2    60   ~ 0
-I2S_MCK
+I2S_MCK#
 Text Label 9500 4800 2    60   ~ 0
-I2S_SD
+I2S_SD#
 Text Label 9500 4600 2    60   ~ 0
-I2S_CK
+I2S_CK#
 Text Label 9500 4500 2    60   ~ 0
-I2S_WS
+I2S_WS#
 Text Label 11100 3650 0    60   ~ 0
 I2S_WS
@@
 	9000 3800 9500 3800
 Wire Wire Line
-	11650 3850 11100 3850
-Wire Wire Line
-	11650 3750 11100 3750
-Wire Wire Line
-	11650 3650 11100 3650
-Wire Wire Line
-	11650 3550 11100 3550
+	10900 3850 11650 3850
+Wire Wire Line
+	10900 3750 11650 3750
+Wire Wire Line
+	10900 3650 11650 3650
+Wire Wire Line
+	10900 3550 11650 3550
 Wire Wire Line
 	9000 5700 9700 5700
@@
 NoConn ~ 9000 6000
 NoConn ~ 2000 6000
+Wire Wire Line
+	10150 3550 10600 3550
+Wire Wire Line
+	10150 3650 10600 3650
+Wire Wire Line
+	10150 3750 10600 3750
+Wire Wire Line
+	10150 3850 10600 3850
+Text Label 10150 3550 0    60   ~ 0
+I2S_MCK#
+Text Label 10150 3650 0    60   ~ 0
+I2S_WS#
+Text Label 10150 3750 0    60   ~ 0
+I2S_CK#
+Text Label 10150 3850 0    60   ~ 0
+I2S_SD#
+$Comp
+L R R?
+U 1 1 56791D61
+P 10750 3550
+F 0 "R?" V 10950 3700 50  0000 C CNN
+F 1 "47" V 10750 3550 50  0000 C CNN
+F 2 "Resistors_SMD:R_0402" V 10680 3550 50  0001 C CNN
+F 3 "" H 10750 3550 50  0000 C CNN
+	1    10750 3550
+	0    -1   -1   0
+$EndComp
+$Comp
+L R R?
+U 1 1 56792500
+P 10750 3650
+F 0 "R?" V 10950 3800 50  0000 C CNN
+F 1 "47" V 10750 3650 50  0000 C CNN
+F 2 "Resistors_SMD:R_0402" V 10680 3650 50  0001 C CNN
+F 3 "" H 10750 3650 50  0000 C CNN
+	1    10750 3650
+	0    -1   -1   0
+$EndComp
+$Comp
+L R R?
+U 1 1 56792684
+P 10750 3750
+F 0 "R?" V 11150 3700 50  0000 C CNN
+F 1 "47" V 10750 3750 50  0000 C CNN
+F 2 "Resistors_SMD:R_0402" V 10680 3750 50  0001 C CNN
+F 3 "" H 10750 3750 50  0000 C CNN
+	1    10750 3750
+	0    -1   -1   0
+$EndComp
+$Comp
+L R R?
+U 1 1 5679280B
+P 10750 3850
+F 0 "R?" V 11150 3800 50  0000 C CNN
+F 1 "47" V 10750 3850 50  0000 C CNN
+F 2 "Resistors_SMD:R_0402" V 10680 3850 50  0001 C CNN
+F 3 "" H 10750 3850 50  0000 C CNN
+	1    10750 3850
+	0    -1   -1   0
+$EndComp
 $EndSCHEMATC

Commit message: version sent to rezonit
modified usb connector pads to smd
Parts:
- added JP101, JP102, JP103, JP104, JP105, JP106: Jumper_NC_Small, Resistors_SMD:R_0603, symbol Jumper_NC_Small
- gave numbers to parts that had none: 4
Connections:
- net GNDA: now also JP101.1, JP102.1, JP105.1, JP106.1
- net GNDD: now also JP101.2, JP102.2, JP103.2, JP104.2
- new net GNDPWR: JP103.1, JP104.1, JP105.2, JP106.2
Changed lines of the file:
@@
 I2S_SD#
 $Comp
-L R R?
+L R R123
 U 1 1 56791D61
 P 10750 3550
-F 0 "R?" V 10950 3700 50  0000 C CNN
+F 0 "R123" V 10950 3700 50  0000 C CNN
 F 1 "47" V 10750 3550 50  0000 C CNN
 F 2 "Resistors_SMD:R_0402" V 10680 3550 50  0001 C CNN
@@
 $EndComp
 $Comp
-L R R?
+L R R124
 U 1 1 56792500
 P 10750 3650
-F 0 "R?" V 10950 3800 50  0000 C CNN
+F 0 "R124" V 10950 3800 50  0000 C CNN
 F 1 "47" V 10750 3650 50  0000 C CNN
 F 2 "Resistors_SMD:R_0402" V 10680 3650 50  0001 C CNN
@@
 $EndComp
 $Comp
-L R R?
+L R R125
 U 1 1 56792684
 P 10750 3750
-F 0 "R?" V 11150 3700 50  0000 C CNN
+F 0 "R125" V 11150 3700 50  0000 C CNN
 F 1 "47" V 10750 3750 50  0000 C CNN
 F 2 "Resistors_SMD:R_0402" V 10680 3750 50  0001 C CNN
@@
 $EndComp
 $Comp
-L R R?
+L R R126
 U 1 1 5679280B
 P 10750 3850
-F 0 "R?" V 11150 3800 50  0000 C CNN
+F 0 "R126" V 11150 3800 50  0000 C CNN
 F 1 "47" V 10750 3850 50  0000 C CNN
 F 2 "Resistors_SMD:R_0402" V 10680 3850 50  0001 C CNN
@@
 	0    -1   -1   0
 $EndComp
+$Comp
+L GNDD #PWR046
+U 1 1 567A8334
+P 15000 2900
+F 0 "#PWR046" H 15000 2650 50  0001 C CNN
+F 1 "GNDD" H 15000 2750 39  0000 C CNN
+F 2 "" H 15000 2900 50  0000 C CNN
+F 3 "" H 15000 2900 50  0000 C CNN
+	1    15000 2900
+	1    0    0    -1
+$EndComp
+$Comp
+L GNDA #PWR047
+U 1 1 567A84B9
+P 15350 2900
+F 0 "#PWR047" H 15350 2650 50  0001 C CNN
+F 1 "GNDA" H 15350 2750 39  0000 C CNN
+F 2 "" H 15350 2900 50  0000 C CNN
+F 3 "" H 15350 2900 50  0000 C CNN
+	1    15350 2900
+	1    0    0    -1
+$EndComp
+$Comp
+L GNDPWR #PWR048
+U 1 1 567A85FA
+P 15750 2900
+F 0 "#PWR048" H 15750 2700 50  0001 C CNN
+F 1 "GNDPWR" H 15750 2770 39  0000 C CNN
+F 2 "" H 15750 2850 50  0000 C CNN
+F 3 "" H 15750 2850 50  0000 C CNN
+	1    15750 2900
+	1    0    0    -1
+$EndComp
+Wire Wire Line
+	15750 2300 15750 2900
+Wire Wire Line
+	15350 2250 15350 2900
+Wire Wire Line
+	15000 2250 15000 2900
+$Comp
+L Jumper_NC_Small JP102
+U 1 1 567ACCA8
+P 15150 2400
+F 0 "JP102" H 15150 2480 50  0000 C CNN
+F 1 "Jumper_NC_Small" H 15160 2340 50  0001 C CNN
+F 2 "Resistors_SMD:R_0603" H 15150 2400 50  0001 C CNN
+F 3 "" H 15150 2400 50  0000 C CNN
+	1    15150 2400
+	-1   0    0    1
+$EndComp
+Wire Wire Line
+	15000 2400 15050 2400
+Connection ~ 15000 2400
+Wire Wire Line
+	15250 2400 15350 2400
+Connection ~ 15350 2400
+$Comp
+L Jumper_NC_Small JP103
+U 1 1 567AE393
+P 15150 2550
+F 0 "JP103" H 15150 2630 50  0000 C CNN
+F 1 "Jumper_NC_Small" H 15160 2490 50  0001 C CNN
+F 2 "Resistors_SMD:R_0603" H 15150 2550 50  0001 C CNN
+F 3 "" H 15150 2550 50  0000 C CNN
+	1    15150 2550
+	-1   0    0    1
+$EndComp
+Wire Wire Line
+	15000 2550 15050 2550
+Connection ~ 15000 2550
+Wire Wire Line
+	15250 2550 15750 2550
+Connection ~ 15750 2550
+Wire Wire Line
+	15350 2450 15450 2450
+Connection ~ 15350 2450
+Wire Wire Line
+	15650 2450 15750 2450
+Connection ~ 15750 2450
+$Comp
+L Jumper_NC_Small JP101
+U 1 1 567B0189
+P 15150 2250
+F 0 "JP101" H 15150 2330 50  0000 C CNN
+F 1 "Jumper_NC_Small" H 15160 2190 50  0001 C CNN
+F 2 "Resistors_SMD:R_0603" H 15150 2250 50  0001 C CNN
+F 3 "" H 15150 2250 50  0000 C CNN
+	1    15150 2250
+	-1   0    0    1
+$EndComp
+Wire Wire Line
+	15000 2250 15050 2250
+Wire Wire Line
+	15350 2250 15250 2250
+$Comp
+L Jumper_NC_Small JP104
+U 1 1 567B2410
+P 15150 2750
+F 0 "JP104" H 15150 2830 50  0000 C CNN
+F 1 "Jumper_NC_Small" H 15160 2690 50  0001 C CNN
+F 2 "Resistors_SMD:R_0603" H 15150 2750 50  0001 C CNN
+F 3 "" H 15150 2750 50  0000 C CNN
+	1    15150 2750
+	-1   0    0    1
+$EndComp
+Wire Wire Line
+	15000 2750 15050 2750
+Connection ~ 15000 2750
+Wire Wire Line
+	15250 2750 15750 2750
+Connection ~ 15750 2750
+$Comp
+L Jumper_NC_Small JP105
+U 1 1 567B3E0C
+P 15550 2300
+F 0 "JP105" H 15550 2380 50  0000 C CNN
+F 1 "Jumper_NC_Small" H 15560 2240 50  0001 C CNN
+F 2 "Resistors_SMD:R_0603" H 15550 2300 50  0001 C CNN
+F 3 "" H 15550 2300 50  0000 C CNN
+	1    15550 2300
+	1    0    0    -1
+$EndComp
+Wire Wire Line
+	15350 2300 15450 2300
+Connection ~ 15350 2300
+Wire Wire Line
+	15650 2300 15750 2300
+$Comp
+L Jumper_NC_Small JP106
+U 1 1 567AE8F5
+P 15550 2450
+F 0 "JP106" H 15550 2530 50  0000 C CNN
+F 1 "Jumper_NC_Small" H 15560 2390 50  0001 C CNN
+F 2 "Resistors_SMD:R_0603" H 15550 2450 50  0001 C CNN
+F 3 "" H 15550 2450 50  0000 C CNN
+	1    15550 2450
+	1    0    0    -1
+$EndComp
 $EndSCHEMATC

Commit message: fixed p-mosfets
Parts:
- R112, R114: value 47K -> 10K
- R113: value 47K -> N/C
Changed lines of the file:
@@
 P 7950 750
 F 0 "R112" V 8050 650 50  0000 C CNN
-F 1 "47K" V 8050 850 50  0000 C CNN
+F 1 "10K" V 8050 850 50  0000 C CNN
 F 2 "Resistors_SMD:R_0805" V 7880 750 50  0001 C CNN
 F 3 "" H 7950 750 50  0000 C CNN
@@
 P 8200 750
 F 0 "R113" V 8300 650 50  0000 C CNN
-F 1 "47K" V 8300 850 50  0000 C CNN
+F 1 "N/C" V 8300 850 50  0000 C CNN
 F 2 "Resistors_SMD:R_0805" V 8130 750 50  0001 C CNN
 F 3 "" H 8200 750 50  0000 C CNN
@@
 P 8450 750
 F 0 "R114" V 8550 650 50  0000 C CNN
-F 1 "47K" V 8550 850 50  0000 C CNN
+F 1 "10K" V 8550 850 50  0000 C CNN
 F 2 "Resistors_SMD:R_0805" V 8380 750 50  0001 C CNN
 F 3 "" H 8450 750 50  0000 C CNN
