File: kicad/_saved_audioout.sch (KiCad schematic (older format))
At the start: 103 parts, among them J301 KATE_3.5MM_6, J302 KATE_3.5MM_6, P301 CONN_02X04, P302 CONN_01X03, Q301 Si2301DS, Q302 IRLML2502, U301 OP275S, U302 OP275S, U303 LM4864, U304 LM4864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

Commit message: circuit fixes
Parts:
- gave numbers to parts that had none: 2
Changed lines of the file:
@@
 $EndComp
 $Comp
-L R R?
+L R R343
 U 1 1 5688629D
 P 3750 10350
-F 0 "R?" V 3850 10350 50  0000 C CNN
+F 0 "R343" V 3850 10350 50  0000 C CNN
 F 1 "20K" V 3650 10350 50  0000 C CNN
 F 2 "Resistors_SMD:R_0805" V 3680 10350 50  0001 C CNN
@@
 	3600 10350 3500 10350
 $Comp
-L R R?
+L R R344
 U 1 1 56887427
 P 3800 12300
-F 0 "R?" V 3900 12300 50  0000 C CNN
+F 0 "R344" V 3900 12300 50  0000 C CNN
 F 1 "20K" V 3700 12300 50  0000 C CNN
 F 2 "Resistors_SMD:R_0805" V 3730 12300 50  0001 C CNN
