File: kicad/megapower.sch (KiCad schematic (older format))
At the start: 51 parts

Commit message: ...
Parts:
- C212, C219: renamed from C?; value 100.0/25V -> 56.0/20V
- C220: renamed from C?; value 100.0/16V -> 56.0/20V
- CON201: renamed from CON?; value BARREL_JACK -> K375A (DJK-02A)
- gave numbers to parts that had none: 46

Commit message: ...
Parts:
- added C? (x2): 0.1, symbol C_Small
Connections:
- wire segments 121 -> 125
Changed lines of the file:
@@
 Text HLabel 1850 3250 1    60   Input ~ 0
 +5VJACK
+$Comp
+L C_Small C?
+U 1 1 5687F839
+P 3500 2400
+F 0 "C?" H 3510 2470 50  0000 L CNN
+F 1 "0.1" H 3510 2320 50  0000 L CNN
+F 2 "" H 3500 2400 50  0000 C CNN
+F 3 "" H 3500 2400 50  0000 C CNN
+	1    3500 2400
+	0    1    1    0
+$EndComp
+$Comp
+L C_Small C?
+U 1 1 5687F911
+P 3500 2550
+F 0 "C?" H 3510 2620 50  0000 L CNN
+F 1 "0.1" H 3510 2470 50  0000 L CNN
+F 2 "" H 3500 2550 50  0000 C CNN
+F 3 "" H 3500 2550 50  0000 C CNN
+	1    3500 2550
+	0    1    1    0
+$EndComp
+$Comp
+L GNDPWR #PWR?
+U 1 1 5687F9C2
+P 3650 2650
+F 0 "#PWR?" H 3650 2450 50  0001 C CNN
+F 1 "GNDPWR" H 3650 2520 50  0000 C CNN
+F 2 "" H 3650 2600 50  0000 C CNN
+F 3 "" H 3650 2600 50  0000 C CNN
+	1    3650 2650
+	1    0    0    -1
+$EndComp
+Wire Wire Line
+	3600 2400 3650 2400
+Wire Wire Line
+	3650 2400 3650 2650
+Wire Wire Line
+	3600 2550 3650 2550
+Connection ~ 3650 2550
+$Comp
+L GNDPWR #PWR?
+U 1 1 5687FE2D
+P 3400 2650
+F 0 "#PWR?" H 3400 2450 50  0001 C CNN
+F 1 "GNDPWR" H 3400 2520 50  0000 C CNN
+F 2 "" H 3400 2600 50  0000 C CNN
+F 3 "" H 3400 2600 50  0000 C CNN
+	1    3400 2650
+	1    0    0    -1
+$EndComp
+Wire Wire Line
+	3400 2400 3400 2650
+Connection ~ 3400 2550
 $EndSCHEMATC

Commit message: ...
Parts:
- removed U203: TPS76333DBV, SOT-23-5, symbol TPS769XX
- added U???: MC33269-SO8, symbol MC33269-SO8
Connections:
- wire segments 125 -> 181
- no-connect marks 2 -> 1
Changed lines of the file:
@@
 LIBS:ad1955
 LIBS:lm4864
+LIBS:mc33269
 LIBS:synth-cache
 EELAYER 25 0
@@
 $EndComp
 $Comp
-L TPS769XX U203
-U 1 1 566ECB9D
-P 3850 3950
-F 0 "U203" H 3600 4250 50  0000 C CNN
-F 1 "TPS76333DBV" H 4000 4250 50  0000 C CNN
-F 2 "SOT-23-5" H 3850 4100 50  0001 C CIN
-F 3 "" H 3850 3950 50  0000 C CNN
-	1    3850 3950
-	1    0    0    -1
-$EndComp
-$Comp
 L C_Small C203
 U 1 1 566ECBA4
@@
 L GNDD #PWR038
 U 1 1 566ECBB2
-P 3850 4250
-F 0 "#PWR038" H 3850 4000 50  0001 C CNN
-F 1 "GNDD" H 3850 4100 50  0000 C CNN
-F 2 "" H 3850 4250 50  0000 C CNN
-F 3 "" H 3850 4250 50  0000 C CNN
-	1    3850 4250
+P 3850 4300
+F 0 "#PWR038" H 3850 4050 50  0001 C CNN
+F 1 "GNDD" H 3850 4150 50  0000 C CNN
+F 2 "" H 3850 4300 50  0000 C CNN
+F 3 "" H 3850 4300 50  0000 C CNN
+	1    3850 4300
 	1    0    0    -1
 $EndComp
@@
 	1    0    0    -1
 $EndComp
-Text Label 1850 3250 3    60   ~ 0
-+5V_UNREG
 $Comp
 L GNDPWR #PWR041
@@
 	1    0    0    -1
 $EndComp
-NoConn ~ 4300 3950
 NoConn ~ 4300 5100
 $Comp
@@
 	3850 950  3950 950
 Wire Wire Line
-	4150 950  5950 950
+	4150 950  5050 950
+Wire Wire Line
+	5050 950  5300 950
+Wire Wire Line
+	5300 950  5950 950
 Wire Wire Line
 	3850 1650 4000 1650
 Wire Wire Line
-	4700 1550 6400 1550
-Wire Wire Line
-	4150 2200 5700 2200
+	4700 1550 5050 1550
+Wire Wire Line
+	5050 1550 5300 1550
+Wire Wire Line
+	5300 1550 6400 1550
+Wire Wire Line
+	4150 2200 4400 2200
+Wire Wire Line
+	4400 2200 4650 2200
+Wire Wire Line
+	4650 2200 5700 2200
 Wire Wire Line
 	4650 2200 4650 2250
@@
 Connection ~ 4650 2200
 Wire Wire Line
-	9300 1350 9650 1350
+	9300 1350 9400 1350
+Wire Wire Line
+	9400 1350 9650 1350
 Wire Wire Line
 	7700 1850 7700 1950
 Wire Wire Line
-	7300 2350 9400 2350
+	7300 2350 7700 2350
+Wire Wire Line
+	7700 2350 8500 2350
+Wire Wire Line
+	8500 2350 9400 2350
 Wire Wire Line
 	7700 2350 7700 2150
@@
 	9400 2350 9400 1850
 Wire Wire Line
-	9300 2800 10150 2800
+	9300 2800 9400 2800
+Wire Wire Line
+	9400 2800 9750 2800
+Wire Wire Line
+	9750 2800 10150 2800
 Wire Wire Line
 	7700 3300 7700 3400
@@
 	7700 3000 7700 2800
 Wire Wire Line
-	7050 3000 7700 3000
+	7050 3000 7300 3000
+Wire Wire Line
+	7300 3000 7700 3000
 Connection ~ 7700 3000
 Wire Wire Line
@@
 Connection ~ 8500 3800
 Wire Wire Line
-	3400 3800 3400 3950
-Connection ~ 3400 3800
-Wire Wire Line
 	3150 3800 3150 3950
 Connection ~ 3150 3800
 Wire Wire Line
-	3150 4150 3150 4250
-Wire Wire Line
-	3150 4250 4600 4250
-Wire Wire Line
-	4300 3800 5150 3800
+	3150 4150 3150 4300
+Wire Wire Line
+	3150 4300 3850 4300
+Wire Wire Line
+	3850 4300 4600 4300
+Wire Wire Line
+	4350 3800 4600 3800
+Wire Wire Line
+	4600 3800 5150 3800
 Wire Wire Line
 	4600 3800 4600 3900
 Connection ~ 4600 3800
 Wire Wire Line
-	4600 4250 4600 4100
-Connection ~ 3850 4250
+	4600 4300 4600 4100
+Connection ~ 3850 4300
 Wire Wire Line
 	3400 4950 3400 5100
@@
 	3150 5300 3150 5400
 Wire Wire Line
-	3150 5400 4600 5400
-Wire Wire Line
-	4300 4950 5150 4950
+	3150 5400 3850 5400
+Wire Wire Line
+	3850 5400 4600 5400
+Wire Wire Line
+	4300 4950 4600 4950
+Wire Wire Line
+	4600 4950 5150 4950
 Wire Wire Line
 	4600 4950 4600 5050
@@
 Connection ~ 3850 5400
 Wire Wire Line
-	3750 6350 3750 6900
-Wire Wire Line
-	4150 6050 5600 6050
-Wire Wire Line
-	4150 7200 5600 7200
-Wire Wire Line
-	3000 6050 3350 6050
-Wire Wire Line
-	3000 7200 3350 7200
+	3750 6350 3750 6650
+Wire Wire Line
+	3750 6650 3750 6900
+Wire Wire Line
+	4150 6050 4250 6050
+Wire Wire Line
+	4250 6050 4750 6050
+Wire Wire Line
+	4750 6050 5250 6050
+Wire Wire Line
+	5250 6050 5600 6050
+Wire Wire Line
+	4150 7200 4250 7200
+Wire Wire Line
+	4250 7200 4750 7200
+Wire Wire Line
+	4750 7200 5250 7200
+Wire Wire Line
+	5250 7200 5600 7200
+Wire Wire Line
+	3000 6050 3200 6050
+Wire Wire Line
+	3200 6050 3350 6050
+Wire Wire Line
+	3000 7200 3200 7200
+Wire Wire Line
+	3200 7200 3350 7200
 Wire Wire Line
 	1750 6050 2400 6050
@@
 Connection ~ 4750 6050
 Wire Wire Line
-	4250 6450 4250 6800
-Wire Wire Line
-	4750 6450 4750 6800
+	4250 6450 4250 6650
+Wire Wire Line
+	4250 6650 4250 6800
+Wire Wire Line
+	4750 6450 4750 6650
+Wire Wire Line
+	4750 6650 4750 6800
 Connection ~ 4250 6650
 Connection ~ 4750 6650
 Wire Wire Line
-	1450 3900 1450 4150
+	1450 3900 1450 4000
+Wire Wire Line
+	1450 4000 1450 4150
 Connection ~ 1450 4000
 Wire Wire Line
-	2800 3800 3400 3800
-Wire Wire Line
-	2900 4950 3400 4950
-Wire Wire Line
-	1450 3800 2200 3800
+	2800 3800 2900 3800
+Wire Wire Line
+	2900 3800 3150 3800
+Wire Wire Line
+	3150 3800 3350 3800
+Wire Wire Line
+	2900 4950 3150 4950
+Wire Wire Line
+	3150 4950 3400 4950
+Wire Wire Line
+	1450 3800 1850 3800
+Wire Wire Line
+	1850 3800 2200 3800
 Wire Wire Line
 	2900 4950 2900 3800
 Connection ~ 2900 3800
 Wire Wire Line
-	7000 1550 7700 1550
-Wire Wire Line
-	5250 6450 5250 6800
+	7000 1550 7050 1550
+Wire Wire Line
+	7050 1550 7300 1550
+Wire Wire Line
+	7300 1550 7700 1550
+Wire Wire Line
+	5250 6450 5250 6650
+Wire Wire Line
+	5250 6650 5250 6800
 Wire Wire Line
 	5250 6250 5250 6050
@@
 Connection ~ 3200 6050
 Wire Wire Line
-	3200 6450 3200 6850
+	3200 6450 3200 6650
+Wire Wire Line
+	3200 6650 3200 6850
 Connection ~ 3200 6650
 Wire Wire Line
@@
 	3850 2200 3950 2200
 Wire Wire Line
-	3200 6650 5850 6650
-Wire Wire Line
-	1000 1900 1500 1900
+	3200 6650 3750 6650
+Wire Wire Line
+	3750 6650 4250 6650
+Wire Wire Line
+	4250 6650 4750 6650
+Wire Wire Line
+	4750 6650 5250 6650
+Wire Wire Line
+	5250 6650 5850 6650
+Wire Wire Line
+	1000 1900 1400 1900
+Wire Wire Line
+	1400 1900 1500 1900
 Connection ~ 1800 2550
 Wire Wire Line
@@
 	1400 1900 1400 2000
 Wire Wire Line
-	1850 3250 1850 3800
+	1850 3450 1850 3800
 Text Label 600  850  0    60   ~ 0
 +5V_UNREG
@@
 Connection ~ 5300 1250
 Wire Wire Line
-	1000 2250 2700 2250
+	1000 2250 2600 2250
+Wire Wire Line
+	2600 2250 2700 2250
 Wire Wire Line
 	7050 3000 7050 1550
 Connection ~ 7050 1550
 Wire Wire Line
-	7300 3800 9750 3800
+	7300 3800 7700 3800
+Wire Wire Line
+	7700 3800 8500 3800
+Wire Wire Line
+	8500 3800 9400 3800
+Wire Wire Line
+	9400 3800 9750 3800
 Text HLabel 1000 1900 0    60   Input ~ 0
 XPULL
@@
 $EndComp
 Wire Wire Line
-	1350 750  1350 1050
+	1350 750  1350 850
+Wire Wire Line
+	1350 850  1350 950
+Wire Wire Line
+	1350 950  1350 1050
 Connection ~ 1350 950
 Connection ~ 1350 850
 Wire Wire Line
-	1950 750  1950 950
+	1950 750  1950 850
+Wire Wire Line
+	1950 850  1950 950
 Connection ~ 1950 850
 $Comp
@@
 	1950 1100 1950 1150
 Wire Wire Line
-	600  850  1350 850
+	600  850  1000 850
+Wire Wire Line
+	1000 850  1350 850
 $Comp
 L CP1_Small C201
@@
 $EndComp
 Wire Wire Line
-	1950 850  2500 850
+	1950 850  2250 850
+Wire Wire Line
+	2250 850  2500 850
 Wire Wire Line
 	2250 850  2250 900
@@
 $EndComp
 Wire Wire Line
-	6550 950  7500 950
+	6550 950  6700 950
+Wire Wire Line
+	6700 950  7500 950
 Wire Wire Line
 	6550 750  6550 650
 Wire Wire Line
-	5950 650  6900 650
+	5950 650  6550 650
+Wire Wire Line
+	6550 650  6900 650
 Wire Wire Line
 	5950 950  5950 650
@@
 Text HLabel 7500 950  2    60   Input ~ 0
 VFEEDBACK
-Text HLabel 1850 3250 1    60   Input ~ 0
+Text HLabel 1850 3450 1    60   Input ~ 0
 +5VJACK
 $Comp
@@
 	3600 2400 3650 2400
 Wire Wire Line
-	3650 2400 3650 2650
+	3650 2400 3650 2550
+Wire Wire Line
+	3650 2550 3650 2650
 Wire Wire Line
 	3600 2550 3650 2550
@@
 $EndComp
 Wire Wire Line
-	3400 2400 3400 2650
+	3400 2400 3400 2550
+Wire Wire Line
+	3400 2550 3400 2650
 Connection ~ 3400 2550
+$Comp
+L MC33269-SO8 U???
+U 1 1 56897419
+P 3850 3950
+F 0 "U???" H 3550 4250 60  0000 C CNN
+F 1 "MC33269-SO8" H 4100 4250 60  0000 C CNN
+F 2 "" H 3950 3600 60  0000 C CNN
+F 3 "" H 3950 3600 60  0000 C CNN
+	1    3850 3950
+	1    0    0    -1
+$EndComp
+Wire Wire Line
+	4350 3800 4350 3900
+Wire Wire Line
+	4350 3900 4350 4000
+Wire Wire Line
+	4350 4000 4350 4100
+Connection ~ 4350 3900
+Connection ~ 4350 4000
+Connection ~ 4350 3800
 $EndSCHEMATC

Commit message: ...
Parts:
- removed U201: LM7812, symbol LM7812
- removed U202: LM7912, symbol LM7912
- added U201: LM78L12ACZ, TO_SOT_Packages_THT:TO-92_Inline_Wide, symbol LM78L12ACZ
- added U202: 79L12, TO_SOT_Packages_THT:TO-92_Inline_Wide, symbol LM7912CT
- C201, C202: footprint (none) -> Capacitors_SMD:c_elec_5x5.3
- C203, C204, C205, C206: footprint (none) -> Capacitors_SMD:C_0805
- C207, C208: renamed from C?; footprint (none) -> Capacitors_SMD:C_0805
- C209: renamed from C207; footprint (none) -> Capacitors_SMD:C_0805
- C210: renamed from C208; footprint (none) -> Capacitors_SMD:C_0805
- C211: renamed from C209; footprint (none) -> Capacitors_SMD:C_0805
- C212: renamed from C210; footprint (none) -> Capacitors_SMD:C_0805
- C213: renamed from C211; footprint (none) -> Capacitors_SMD:C_0805
- C214: renamed from C212; footprint (none) -> Capacitors_ThroughHole:C_Radial_D6.3_L11.2_P2.5
- C215: renamed from C213; footprint (none) -> Capacitors_SMD:c_elec_6.3x7.7
- C216: renamed from C214; footprint (none) -> Capacitors_SMD:c_elec_6.3x7.7
- C217: renamed from C215; footprint (none) -> Capacitors_SMD:C_0603
- C218: renamed from C216; footprint (none) -> Capacitors_SMD:C_0603
- C219: renamed from C217; footprint (none) -> Capacitors_SMD:c_elec_6.3x7.7
- C220: renamed from C218; footprint (none) -> Capacitors_SMD:c_elec_6.3x7.7
- C221: renamed from C219; footprint (none) -> Capacitors_ThroughHole:C_Radial_D6.3_L11.2_P2.5
- C222: renamed from C220; footprint (none) -> Capacitors_ThroughHole:C_Radial_D6.3_L11.2_P2.5
- C223: renamed from C221; footprint (none) -> Capacitors_SMD:C_0805
- C224: renamed from C222; footprint (none) -> Capacitors_SMD:C_0805
- C225: renamed from C223; footprint (none) -> Capacitors_SMD:C_0805
- C226: renamed from C224; footprint (none) -> Capacitors_SMD:C_0805
- C227: renamed from C225; footprint (none) -> Capacitors_SMD:C_0805
- C228: renamed from C226; footprint (none) -> Capacitors_SMD:C_0805
- C229: renamed from C227; value 10.0/10V -> 22.0/10V; footprint (none) -> Capacitors_Tantalum_SMD:TantalC_SizeC_EIA-6032_Reflow
- CON201: footprint (none) -> Connect:BARREL_JACK
- D201, D202, D203: footprint (none) -> Diodes_SMD:SMB_Standard
- D204: footprint (none) -> TO_SOT_Packages_SMD:SOT-23
- L201, L202, L203, L204: footprint (none) -> Choke_SMD:Choke_SMD_6.3x6.3_H3
- Q201: footprint MICRO8 -> Housings_SOIC:SOIC-8_3.9x4.9mm_Pitch1.27mm
- Q202: footprint SO-8 -> Power_Integrations:SO-8
- R201, R202, R203, R204, R205: footprint (none) -> Resistors_SMD:R_0805
- T201: footprint (none) -> Transformers_SMPS_ThroughHole:Coilcraft-Q4434-B_Rhombus-T1311
- U203: renamed from U???; footprint (none) -> Housings_SOIC:SOIC-8_3.9x4.9mm_Pitch1.27mm
- U204: footprint SOT-23-5 -> TO_SOT_Packages_SMD:SOT-23-5
- U205, U206: footprint (none) -> TO_SOT_Packages_SMD:SOT-23-5
Connections:
- wire segments 181 -> 126

Commit message: gruuuu
Connections:
- net +5V_UNREG is gone; now on net +5VJACK: C201.1, Q201.5 (D), Q201.6 (D), Q201.7 (D), Q201.8 (D)
- net +15V: no longer D204.2 (K)
- net +3V3D_CPU: now also D204.2 (K)
Changed lines of the file:
@@
 Wire Wire Line
 	1850 3450 1850 3800
-Text Label 600  850  0    60   ~ 0
-+5V_UNREG
 $Comp
 L C_Small C218
@@
 F 0 "Q201" H 1450 1250 50  0000 L CNN
 F 1 "FDS6675" H 1450 700 50  0000 L CNN
-F 2 "Housings_SOIC:SOIC-8_3.9x4.9mm_Pitch1.27mm" H 1650 1150 50  0000 C CIN
+F 2 "Housings_SOIC:SOIC-8_3.9x4.9mm_Pitch1.27mm" H 1650 1150 50  0001 C CIN
 F 3 "" V 1650 950 50  0000 L CNN
 	1    1650 950
@@
 	1950 1100 1950 1150
 Wire Wire Line
-	600  850  1350 850
+	950  850  1350 850
 $Comp
 L CP1_Small C201
@@
 	6550 750  6550 650
 Wire Wire Line
-	5950 650  6900 650
-Wire Wire Line
 	5950 950  5950 650
-Connection ~ 6550 650
 Wire Wire Line
 	6550 1150 6550 1250
@@
 	1    0    0    -1
 $EndComp
+Wire Wire Line
+	5950 650  6550 650
+Text GLabel 7100 650  2    60   Input ~ 0
++3V3D_CPU
+Wire Wire Line
+	6900 650  7100 650
+Text HLabel 950  850  0    60   Input ~ 0
++5VJACK
 $EndSCHEMATC

Commit message: drc ok large vias
Connections:
- net GNDPWR: no longer C207.1, C207.2, C208.1, C208.2
- no-connect marks 1 -> 5
Other:
- moved on the sheet: C208
Changed lines of the file:
@@
 L C_Small C208
 U 1 1 5687F911
-P 3500 2550
-F 0 "C208" H 3510 2620 50  0000 L CNN
-F 1 "0.1" H 3510 2470 50  0000 L CNN
-F 2 "Capacitors_SMD:C_0805" H 3500 2550 50  0001 C CNN
-F 3 "" H 3500 2550 50  0000 C CNN
-	1    3500 2550
+P 3500 2650
+F 0 "C208" H 3510 2720 50  0000 L CNN
+F 1 "0.1" H 3510 2570 50  0000 L CNN
+F 2 "Capacitors_SMD:C_0805" H 3500 2650 50  0001 C CNN
+F 3 "" H 3500 2650 50  0000 C CNN
+	1    3500 2650
 	0    1    1    0
 $EndComp
-$Comp
-L GNDPWR #PWR062
-U 1 1 5687F9C2
-P 3650 2650
-F 0 "#PWR062" H 3650 2450 50  0001 C CNN
-F 1 "GNDPWR" H 3650 2520 50  0000 C CNN
-F 2 "" H 3650 2600 50  0000 C CNN
-F 3 "" H 3650 2600 50  0000 C CNN
-	1    3650 2650
-	1    0    0    -1
-$EndComp
-Wire Wire Line
-	3600 2400 3650 2400
-Wire Wire Line
-	3650 2400 3650 2650
-Wire Wire Line
-	3600 2550 3650 2550
-Connection ~ 3650 2550
-$Comp
-L GNDPWR #PWR063
-U 1 1 5687FE2D
-P 3400 2650
-F 0 "#PWR063" H 3400 2450 50  0001 C CNN
-F 1 "GNDPWR" H 3400 2520 50  0000 C CNN
-F 2 "" H 3400 2600 50  0000 C CNN
-F 3 "" H 3400 2600 50  0000 C CNN
-	1    3400 2650
-	1    0    0    -1
-$EndComp
-Wire Wire Line
-	3400 2400 3400 2650
-Connection ~ 3400 2550
 $Comp
 L MC33269-SO8 U203
@@
 Connection ~ 4350 3800
 $Comp
-L PWR_FLAG #FLG064
+L PWR_FLAG #FLG062
 U 1 1 56A5C59A
 P 7300 1450
-F 0 "#FLG064" H 7300 1545 50  0001 C CNN
+F 0 "#FLG062" H 7300 1545 50  0001 C CNN
 F 1 "PWR_FLAG" H 7300 1650 50  0000 C CNN
 F 2 "" H 7300 1450 50  0000 C CNN
@@
 $EndComp
 $Comp
-L PWR_FLAG #FLG065
+L PWR_FLAG #FLG063
 U 1 1 56A5EB02
 P 2700 4500
-F 0 "#FLG065" H 2700 4595 50  0001 C CNN
+F 0 "#FLG063" H 2700 4595 50  0001 C CNN
 F 1 "PWR_FLAG" H 2700 4700 50  0000 C CNN
 F 2 "" H 2700 4500 50  0000 C CNN
@@
 Connection ~ 2900 4500
 $Comp
-L PWR_FLAG #FLG066
+L PWR_FLAG #FLG064
 U 1 1 56A5F554
 P 3200 5950
-F 0 "#FLG066" H 3200 6045 50  0001 C CNN
+F 0 "#FLG064" H 3200 6045 50  0001 C CNN
 F 1 "PWR_FLAG" H 3200 6150 50  0000 C CNN
 F 2 "" H 3200 5950 50  0000 C CNN
@@
 $EndComp
 $Comp
-L PWR_FLAG #FLG067
+L PWR_FLAG #FLG065
 U 1 1 56A5FD2B
 P 3200 7350
-F 0 "#FLG067" H 3200 7445 50  0001 C CNN
+F 0 "#FLG065" H 3200 7445 50  0001 C CNN
 F 1 "PWR_FLAG" H 3200 7550 50  0000 C CNN
 F 2 "" H 3200 7350 50  0000 C CNN
@@
 Text HLabel 950  850  0    60   Input ~ 0
 +5VJACK
+NoConn ~ 3600 2400
+NoConn ~ 3600 2650
+NoConn ~ 3400 2650
+NoConn ~ 3400 2400
 $EndSCHEMATC
