File: kicad/megapower.sch (KiCad schematic (older format))
At the start: 52 parts, among them CON201 K375A (DJK-02A), Q201 FDS6675, Q202 IRF7313PBF, T201 TRANS_CUSTOM, U201 LM78L12ACZ, U202 79L12, U203 MC33269-SO8, U204 TPS76333DBV, U205 LP2985LV, U206 LP2985LV

Commit message: version sent to rezonit
modified usb connector pads to smd
Parts:
- added +12V201, +3V3A201, +3V3D201, +5VA201, +5VD201, -12V201, FEEDBACK201, GNDA1, W202, W203, W204: TST, Connect:PINTST, symbol TEST_1P
- added +15V201: TST+15V, Connect:PINTST, symbol TEST_1P
- added -15V201: TST-15V, Connect:PINTST, symbol TEST_1P
Connections:
- net +12VOPA: now also +12V201.1
- net +15V: now also +15V201.1
- net +3V3A_CPU: now also +3V3A201.1
- net +3V3D_CPU: now also +3V3D201.1
- net +5VA_DAC: now also +5VA201.1
- net +5VD_DAC: now also +5VD201.1
- net -12VOPA: now also -12V201.1
- net -15V: now also -15V201.1
- net GNDA: now also GNDA1.1
- net GNDPWR: now also W204.1
- net VFEEDBACK: now also FEEDBACK201.1
- net XPULL: now also W202.1
- net XPUSH: now also W203.1
- net at R203.1, T201.2 (PM): now also T201.3
Changed lines of the file:
@@
 $EndComp
 $Comp
-L GNDPWR #PWR046
+L GNDPWR #PWR049
 U 1 1 566E59F2
 P 3000 2650
-F 0 "#PWR046" H 3000 2450 50  0001 C CNN
+F 0 "#PWR049" H 3000 2450 50  0001 C CNN
 F 1 "GNDPWR" H 3000 2520 50  0000 C CNN
 F 2 "" H 3000 2600 50  0000 C CNN
@@
 $EndComp
 $Comp
-L GNDPWR #PWR047
+L GNDPWR #PWR050
 U 1 1 566E5A97
 P 1800 2550
-F 0 "#PWR047" H 1800 2350 50  0001 C CNN
+F 0 "#PWR050" H 1800 2350 50  0001 C CNN
 F 1 "GNDPWR" H 1800 2420 50  0000 C CNN
 F 2 "" H 1800 2500 50  0000 C CNN
@@
 $EndComp
 $Comp
-L GNDPWR #PWR048
+L GNDPWR #PWR051
 U 1 1 566E7760
 P 4000 1650
-F 0 "#PWR048" H 4000 1450 50  0001 C CNN
+F 0 "#PWR051" H 4000 1450 50  0001 C CNN
 F 1 "GNDPWR" H 4000 1520 50  0000 C CNN
 F 2 "" H 4000 1600 50  0000 C CNN
@@
 $EndComp
 $Comp
-L GNDPWR #PWR049
+L GNDPWR #PWR052
 U 1 1 566E9409
 P 4650 2500
-F 0 "#PWR049" H 4650 2300 50  0001 C CNN
+F 0 "#PWR052" H 4650 2300 50  0001 C CNN
 F 1 "GNDPWR" H 4650 2370 50  0000 C CNN
 F 2 "" H 4650 2450 50  0000 C CNN
@@
 $EndComp
 $Comp
-L GNDPWR #PWR050
+L GNDPWR #PWR053
 U 1 1 566E987F
 P 5300 1850
-F 0 "#PWR050" H 5300 1650 50  0001 C CNN
+F 0 "#PWR053" H 5300 1650 50  0001 C CNN
 F 1 "GNDPWR" H 5300 1720 50  0000 C CNN
 F 2 "" H 5300 1800 50  0000 C CNN
@@
 $EndComp
 $Comp
-L GNDPWR #PWR051
+L GNDPWR #PWR054
 U 1 1 566E98CF
 P 5300 1250
-F 0 "#PWR051" H 5300 1050 50  0001 C CNN
+F 0 "#PWR054" H 5300 1050 50  0001 C CNN
 F 1 "GNDPWR" H 5300 1120 50  0000 C CNN
 F 2 "" H 5300 1200 50  0000 C CNN
@@
 +5VA_DAC
 $Comp
-L GNDD #PWR052
+L GNDD #PWR055
 U 1 1 566ECB60
 P 8500 2350
-F 0 "#PWR052" H 8500 2100 50  0001 C CNN
+F 0 "#PWR055" H 8500 2100 50  0001 C CNN
 F 1 "GNDD" H 8500 2200 50  0000 C CNN
 F 2 "" H 8500 2350 50  0000 C CNN
@@
 $EndComp
 $Comp
-L GNDA #PWR053
+L GNDA #PWR056
 U 1 1 566ECB66
 P 8500 3800
-F 0 "#PWR053" H 8500 3550 50  0001 C CNN
+F 0 "#PWR056" H 8500 3550 50  0001 C CNN
 F 1 "GNDA" H 8500 3650 50  0000 C CNN
 F 2 "" H 8500 3800 50  0000 C CNN
@@
 $EndComp
 $Comp
-L GNDD #PWR054
+L GNDD #PWR057
 U 1 1 566ECBB2
 P 3850 4300
-F 0 "#PWR054" H 3850 4050 50  0001 C CNN
+F 0 "#PWR057" H 3850 4050 50  0001 C CNN
 F 1 "GNDD" H 3850 4150 50  0000 C CNN
 F 2 "" H 3850 4300 50  0000 C CNN
@@
 +3V3A_CPU
 $Comp
-L GNDA #PWR055
+L GNDA #PWR058
 U 1 1 566ECBCF
 P 3850 5400
-F 0 "#PWR055" H 3850 5150 50  0001 C CNN
+F 0 "#PWR058" H 3850 5150 50  0001 C CNN
 F 1 "GNDA" H 3850 5250 50  0000 C CNN
 F 2 "" H 3850 5400 50  0000 C CNN
@@
 -12VOPA
 $Comp
-L GNDA #PWR056
+L GNDA #PWR059
 U 1 1 566ECC1D
 P 5850 6650
-F 0 "#PWR056" H 5850 6400 50  0001 C CNN
+F 0 "#PWR059" H 5850 6400 50  0001 C CNN
 F 1 "GNDA" H 5850 6500 50  0000 C CNN
 F 2 "" H 5850 6650 50  0000 C CNN
@@
 $EndComp
 $Comp
-L GNDPWR #PWR057
+L GNDPWR #PWR060
 U 1 1 566ECC33
 P 1450 4150
-F 0 "#PWR057" H 1450 3950 50  0001 C CNN
+F 0 "#PWR060" H 1450 3950 50  0001 C CNN
 F 1 "GNDPWR" H 1450 4020 50  0000 C CNN
 F 2 "" H 1450 4100 50  0000 C CNN
@@
 Connection ~ 1800 2550
 Wire Wire Line
-	1800 2550 1400 2550
+	1400 2550 1950 2550
 Connection ~ 1400 1900
 Wire Wire Line
@@
 Connection ~ 1950 850
 $Comp
-L GNDPWR #PWR058
+L GNDPWR #PWR061
 U 1 1 5673783D
 P 1950 1150
-F 0 "#PWR058" H 1950 950 50  0001 C CNN
+F 0 "#PWR061" H 1950 950 50  0001 C CNN
 F 1 "GNDPWR" H 1950 1020 39  0001 C CNN
 F 2 "" H 1950 1100 50  0000 C CNN
@@
 	1000 1100 1000 1150
 $Comp
-L GNDPWR #PWR059
+L GNDPWR #PWR062
 U 1 1 56738083
 P 1000 1150
-F 0 "#PWR059" H 1000 950 50  0001 C CNN
+F 0 "#PWR062" H 1000 950 50  0001 C CNN
 F 1 "GNDPWR" H 1000 1020 39  0001 C CNN
 F 2 "" H 1000 1100 50  0000 C CNN
@@
 	2250 850  2250 900
 $Comp
-L GNDPWR #PWR060
+L GNDPWR #PWR063
 U 1 1 567382F5
 P 2250 1150
-F 0 "#PWR060" H 2250 950 50  0001 C CNN
+F 0 "#PWR063" H 2250 950 50  0001 C CNN
 F 1 "GNDPWR" H 2250 1020 39  0001 C CNN
 F 2 "" H 2250 1100 50  0000 C CNN
@@
 $EndComp
 $Comp
-L GNDPWR #PWR061
+L GNDPWR #PWR064
 U 1 1 567400B8
 P 6900 1250
-F 0 "#PWR061" H 6900 1050 50  0001 C CNN
+F 0 "#PWR064" H 6900 1050 50  0001 C CNN
 F 1 "GNDPWR" H 6900 1120 50  0001 C CNN
 F 2 "" H 6900 1200 50  0000 C CNN
@@
 Connection ~ 4350 3800
 $Comp
-L PWR_FLAG #FLG062
+L PWR_FLAG #FLG065
 U 1 1 56A5C59A
 P 7300 1450
-F 0 "#FLG062" H 7300 1545 50  0001 C CNN
+F 0 "#FLG065" H 7300 1545 50  0001 C CNN
 F 1 "PWR_FLAG" H 7300 1650 50  0000 C CNN
 F 2 "" H 7300 1450 50  0000 C CNN
@@
 $EndComp
 $Comp
-L PWR_FLAG #FLG063
+L PWR_FLAG #FLG066
 U 1 1 56A5EB02
 P 2700 4500
-F 0 "#FLG063" H 2700 4595 50  0001 C CNN
+F 0 "#FLG066" H 2700 4595 50  0001 C CNN
 F 1 "PWR_FLAG" H 2700 4700 50  0000 C CNN
 F 2 "" H 2700 4500 50  0000 C CNN
@@
 Connection ~ 2900 4500
 $Comp
-L PWR_FLAG #FLG064
+L PWR_FLAG #FLG067
 U 1 1 56A5F554
 P 3200 5950
-F 0 "#FLG064" H 3200 6045 50  0001 C CNN
+F 0 "#FLG067" H 3200 6045 50  0001 C CNN
 F 1 "PWR_FLAG" H 3200 6150 50  0000 C CNN
 F 2 "" H 3200 5950 50  0000 C CNN
@@
 $EndComp
 $Comp
-L PWR_FLAG #FLG065
+L PWR_FLAG #FLG068
 U 1 1 56A5FD2B
 P 3200 7350
-F 0 "#FLG065" H 3200 7445 50  0001 C CNN
+F 0 "#FLG068" H 3200 7445 50  0001 C CNN
 F 1 "PWR_FLAG" H 3200 7550 50  0000 C CNN
 F 2 "" H 3200 7350 50  0000 C CNN
@@
 NoConn ~ 3400 2650
 NoConn ~ 3400 2400
+$Comp
+L TEST_1P +15V201
+U 1 1 5679A488
+P 2100 6050
+F 0 "+15V201" H 2100 6320 50  0000 C CNN
+F 1 "TST+15V" H 2100 6250 50  0000 C CNN
+F 2 "Connect:PINTST" H 2300 6050 50  0001 C CNN
+F 3 "" H 2300 6050 50  0000 C CNN
+	1    2100 6050
+	1    0    0    -1
+$EndComp
+Connection ~ 2100 6050
+$Comp
+L TEST_1P -15V201
+U 1 1 5679B500
+P 2100 7200
+F 0 "-15V201" H 2100 7470 50  0000 C CNN
+F 1 "TST-15V" H 2100 7400 50  0000 C CNN
+F 2 "Connect:PINTST" H 2300 7200 50  0001 C CNN
+F 3 "" H 2300 7200 50  0000 C CNN
+	1    2100 7200
+	1    0    0    -1
+$EndComp
+Connection ~ 2100 7200
+$Comp
+L TEST_1P +12V201
+U 1 1 5679C407
+P 5450 6050
+F 0 "+12V201" H 5450 6320 50  0000 C CNN
+F 1 "TST" H 5450 6250 50  0000 C CNN
+F 2 "Connect:PINTST" H 5650 6050 50  0001 C CNN
+F 3 "" H 5650 6050 50  0000 C CNN
+	1    5450 6050
+	1    0    0    -1
+$EndComp
+Connection ~ 5450 6050
+$Comp
+L TEST_1P -12V201
+U 1 1 5679C596
+P 5450 7200
+F 0 "-12V201" H 5450 7470 50  0000 C CNN
+F 1 "TST" H 5450 7400 50  0000 C CNN
+F 2 "Connect:PINTST" H 5650 7200 50  0001 C CNN
+F 3 "" H 5650 7200 50  0000 C CNN
+	1    5450 7200
+	-1   0    0    1
+$EndComp
+Connection ~ 5450 7200
+$Comp
+L TEST_1P +3V3A201
+U 1 1 5679CD8A
+P 5000 4950
+F 0 "+3V3A201" H 5000 5220 50  0000 C CNN
+F 1 "TST" H 5000 5150 50  0000 C CNN
+F 2 "Connect:PINTST" H 5200 4950 50  0001 C CNN
+F 3 "" H 5200 4950 50  0000 C CNN
+	1    5000 4950
+	1    0    0    -1
+$EndComp
+Connection ~ 5000 4950
+$Comp
+L TEST_1P +3V3D201
+U 1 1 5679CE82
+P 5000 3800
+F 0 "+3V3D201" H 5000 4070 50  0000 C CNN
+F 1 "TST" H 5000 4000 50  0000 C CNN
+F 2 "Connect:PINTST" H 5200 3800 50  0001 C CNN
+F 3 "" H 5200 3800 50  0000 C CNN
+	1    5000 3800
+	1    0    0    -1
+$EndComp
+Connection ~ 5000 3800
+$Comp
+L TEST_1P +5VD201
+U 1 1 5679DE25
+P 10000 1350
+F 0 "+5VD201" H 10000 1620 50  0000 C CNN
+F 1 "TST" H 10000 1550 50  0000 C CNN
+F 2 "Connect:PINTST" H 10200 1350 50  0001 C CNN
+F 3 "" H 10200 1350 50  0000 C CNN
+	1    10000 1350
+	1    0    0    -1
+$EndComp
+$Comp
+L TEST_1P +5VA201
+U 1 1 5679DF5B
+P 10000 2800
+F 0 "+5VA201" H 10000 3070 50  0000 C CNN
+F 1 "TST" H 10000 3000 50  0000 C CNN
+F 2 "Connect:PINTST" H 10200 2800 50  0001 C CNN
+F 3 "" H 10200 2800 50  0000 C CNN
+	1    10000 2800
+	1    0    0    -1
+$EndComp
+Connection ~ 10000 2800
+Connection ~ 10000 1350
+$Comp
+L TEST_1P FEEDBACK201
+U 1 1 5679F66F
+P 7400 850
+F 0 "FEEDBACK201" H 7400 1120 50  0000 C CNN
+F 1 "TST" H 7400 1050 50  0000 C CNN
+F 2 "Connect:PINTST" H 7600 850 50  0001 C CNN
+F 3 "" H 7600 850 50  0000 C CNN
+	1    7400 850
+	0    -1   -1   0
+$EndComp
+Wire Wire Line
+	7400 850  7400 950
+Connection ~ 7400 950
+$Comp
+L TEST_1P W202
+U 1 1 567A0BE8
+P 1200 1900
+F 0 "W202" H 1200 2170 50  0000 C CNN
+F 1 "TST" H 1200 2100 50  0000 C CNN
+F 2 "Connect:PINTST" H 1400 1900 50  0001 C CNN
+F 3 "" H 1400 1900 50  0000 C CNN
+	1    1200 1900
+	1    0    0    -1
+$EndComp
+Connection ~ 1200 1900
+$Comp
+L TEST_1P W203
+U 1 1 567A1272
+P 1200 2250
+F 0 "W203" H 1200 2520 50  0000 C CNN
+F 1 "TST" H 1200 2450 50  0000 C CNN
+F 2 "Connect:PINTST" H 1400 2250 50  0001 C CNN
+F 3 "" H 1400 2250 50  0000 C CNN
+	1    1200 2250
+	1    0    0    -1
+$EndComp
+Connection ~ 1200 2250
+$Comp
+L TEST_1P W204
+U 1 1 567A2D0A
+P 1950 2550
+F 0 "W204" H 1950 2820 50  0000 C CNN
+F 1 "TST" H 1950 2750 50  0000 C CNN
+F 2 "Connect:PINTST" H 2150 2550 50  0001 C CNN
+F 3 "" H 2150 2550 50  0000 C CNN
+	1    1950 2550
+	1    0    0    -1
+$EndComp
+$Comp
+L TEST_1P GNDA1
+U 1 1 567BD11D
+P 9150 3800
+F 0 "GNDA1" H 9150 4070 50  0000 C CNN
+F 1 "TST" H 9150 4000 50  0000 C CNN
+F 2 "Connect:PINTST" H 9350 3800 50  0001 C CNN
+F 3 "" H 9350 3800 50  0000 C CNN
+	1    9150 3800
+	1    0    0    -1
+$EndComp
+Connection ~ 9150 3800
+Connection ~ 2950 1650
 $EndSCHEMATC

Commit message: circuit fixes
Other:
- note added: "Bifilar primary windings: 8+8\nSecondary: 34+34 for -15/+15\n17 for +7.5"
- note removed: "Bifilar primary windings"
Changed lines of the file:
@@
 	0    1    1    0
 $EndComp
-Text Notes 3100 1300 0    39   ~ 0
-Bifilar primary windings
+Text Notes 2850 1250 0    39   ~ 0
+Bifilar primary windings: 8+8\nSecondary: 34+34 for -15/+15\n17 for +7.5
 $Comp
 L D_Small D202
